Commit message: working on urdf

File: src/deepdrive_description/urdf/camera_wide.xacro (robot description, xacro)
@@ -30,5 +30,5 @@
         <link name="${mount_point}_optical_frame"/>
         <gazebo reference="${mount_point}_link">
-            <material>Gazebo/White</material>
+            <!-- <material>Gazebo/White</material> -->
             <sensor type="camera" name="${mount_point}">
                 <pose>0 0 0 0 0 0</pose>

File: src/deepdrive_description/urdf/deepdrive_deepdrive.xacro (robot description, xacro)
@@ -3,4 +3,5 @@
   xmlns:xacro="http://ros.org/wiki/xacro">
   <xacro:property name="wheel_base" value="0.175" />
+  <xacro:property name="wheel_radius" value="0.035" />
   <xacro:include filename="$(find deepdrive_description)/urdf/common_properties.xacro"/>
   <xacro:include filename="$(find deepdrive_description)/urdf/wheels.xacro"/>
@@ -31,8 +32,11 @@
     </inertial>
   </link>
-  <xacro:wheel name="front_right" lr="1" fb="1" wheel_base="${wheel_base}" />
-  <xacro:wheel name="back_right" lr="1" fb="-1" wheel_base="${wheel_base}" />
-  <xacro:wheel name="front_left" lr="-1" fb="-1" wheel_base="${wheel_base}" />
-  <xacro:wheel name="back_left" lr="-1" fb="1" wheel_base="${wheel_base}" />
+  <gazebo reference="base_link">
+    <material>Gazebo/Grey</material>
+  </gazebo>
+  <xacro:wheel name="front_right" lr="1" fb="1" wheel_base="${wheel_base}" wheel_radius="${wheel_radius}" />
+  <xacro:wheel name="back_right" lr="1" fb="-1" wheel_base="${wheel_base}" wheel_radius="${wheel_radius}" />
+  <xacro:wheel name="front_left" lr="-1" fb="-1" wheel_base="${wheel_base}" wheel_radius="${wheel_radius}" />
+  <xacro:wheel name="back_left" lr="-1" fb="1" wheel_base="${wheel_base}" wheel_radius="${wheel_radius}" />
   <!-- <joint name="imu_joint" type="fixed">
     <parent link="base_link"/>
@@ -50,3 +54,49 @@
   <xacro:include filename="$(find deepdrive_description)/urdf/lidar.xacro" />
   <xacro:include filename="$(find deepdrive_description)/urdf/camera.xacro" />
+  <gazebo>
+    <plugin name='diff_drive' filename='libgazebo_ros_diff_drive.so'>
+      <!-- Wheel Information -->
+      <num_wheel_pairs>2</num_wheel_pairs>
+      <left_joint>wheel_front_left_joint</left_joint>
+      <right_joint>wheel_front_right_joint</right_joint>
+      <left_joint>wheel_back_left_joint</left_joint>
+      <right_joint>wheel_back_right_joint</right_joint>
+      <wheel_separation>${wheel_base}</wheel_separation>
+      <wheel_diameter>${wheel_radius*2}</wheel_diameter>
+      <!-- Limits -->
+      <max_wheel_torque>200</max_wheel_torque>
+      <max_wheel_acceleration>10.0</max_wheel_acceleration>
+      <!-- Output -->
+      <odometry_frame>odom</odometry_frame>
+      <robot_base_frame>base_footprint</robot_base_frame>
+      <publish_odom>true</publish_odom>
+      <publish_odom_tf>true</publish_odom_tf>
+      <publish_wheel_tf>true</publish_wheel_tf>
+         <!-- <ros>
+        <namespace>/demo</namespace>
+        <remapping>cmd_vel:=cmd_demo</remapping>
+        <remapping>odom:=odom_demo</remapping>
+      </ros> -->
+      <!-- <updateRate>100.0</updateRate>
+      <robotNamespace>/</robotNamespace>
+      <leftFrontJoint>wheel_front_left_joint</leftFrontJoint>
+      <rightFrontJoint>wheel_front_right_joint</rightFrontJoint>
+      <leftRearJoint>wheel_back_left_joint</leftRearJoint>
+      <rightRearJoint>wheel_back_right_joint</rightRearJoint>
+      <wheelSeparation>${wheel_base}</wheelSeparation>
+      <wheelDiameter>${wheel_radius*2}</wheelDiameter>
+      <robotBaseFrame>base_link</robotBaseFrame>
+      <torque>20</torque>
+      <topicName>cmd_vel</topicName>
+      <broadcastTF>true</broadcastTF>
+      <num_wheel_pairs>2</num_wheel_pairs>
+      <max_wheel_torque>20</max_wheel_torque>
+      <max_wheel_acceleration>1.0</max_wheel_acceleration>
+      <odometry_frame>odom</odometry_frame>
+      <robot_base_frame>base_link</robot_base_frame>
+      <publish_odom>true</publish_odom>
+      <publish_odom_tf>true</publish_odom_tf>
+      <publish_wheel_tf>true</publish_wheel_tf> -->
+    </plugin>
+  </gazebo>
 </robot>

File: src/deepdrive_description/urdf/oakdlite.xacro (robot description, xacro)
@@ -71,5 +71,5 @@
     <link name="${mount_point}_depth_frame"/>
     <gazebo reference="${mount_point}_link">
-      <material>Gazebo/White</material>
+      <material>Gazebo/Black</material>
       <sensor name="${mount_point}_depth" type="depth">
         <pose>0.01233 -0.03 .01878 0 0 0</pose>

File: src/deepdrive_description/urdf/wheels.xacro (robot description, xacro)
@@ -2,13 +2,12 @@
 <robot name="xacro_properties"
     xmlns:xacro="http://ros.org/wiki/xacro">
-    <xacro:property name="wheel_radius" value="0.035" />
     <xacro:property name="wheel_thickness" value="0.025" />
     <xacro:property name="wheel_front_offset" value="-.13" />
-    <xacro:macro name="wheel" params="lr fb name wheel_base">
+    <xacro:macro name="wheel" params="lr fb name wheel_base wheel_radius">
         <joint name="wheel_${name}_joint" type="continuous">
             <parent link="base_link"/>
             <child link="wheel_${name}_link"/>
             <origin xyz="${wheel_front_offset/2 + (fb * (wheel_base / 2))} ${-lr * wheel_base/2} 0.0" rpy="0 0 ${lr*1.57}"/>
-            <axis xyz="1 0 0"/>
+            <axis xyz="${-1*lr} 0 0"/>
         </joint>
         <link name="wheel_${name}_link">
@@ -32,4 +31,7 @@
             </inertial>
         </link>
+        <gazebo reference="wheel_${name}_link">
+            <material>Gazebo/Blue</material>
+        </gazebo>
         <joint name="tire_${name}_joint" type="fixed">
             <parent link="wheel_${name}_link"/>
@@ -58,4 +60,7 @@
             </inertial>
         </link>
+        <gazebo reference="tire_${name}_link">
+            <material>Gazebo/Black</material>
+        </gazebo>
     </xacro:macro>
 </robot>
