Commit message: Localization started

File: src/deepdrive_description/urdf/deepdrive_deepdrive.urdf (robot description, URDF)
Before this commit: robot deepdrive_deepdrive, 13 links, 12 joints
Links:
- link camera_link: geometry collision box size=0.012 0.132 0.020; visual mesh filename=package://depthai_descriptions/urdf/models/OAK-D-LITE.stl

Commit message: Manual focus is working

File: src/deepdrive_description/urdf/deepdrive_deepdrive.urdf (robot description, URDF)
Before this commit: robot deepdrive_deepdrive, 13 links, 12 joints
Links:
- added link oak
Joints:
- added joint oak_joint: type fixed, parent base_link, child oak, origin xyz=0.0 0 0.068 rpy=0 0 0

Commit message: Updated urdf

File: src/deepdrive_description/urdf/deepdrive_deepdrive.urdf (robot description, URDF)
Before this commit: robot deepdrive_deepdrive, 14 links, 13 joints
Links:
- removed link caster_back_left_link
- removed link caster_back_right_link
- added link tire_left_link, mass 2.8498940e-02; collision cylinder length=0.018 radius=0.033; visual mesh filename=package://deepdrive_description/meshes/wheels/tire.stl scale=1 1 1
- added link tire_left_rear_link, mass 2.8498940e-02; collision cylinder length=0.018 radius=0.033; visual mesh filename=package://deepdrive_description/meshes/wheels/tire.stl scale=1 1 1
- added link tire_right_link, mass 2.8498940e-02; collision cylinder length=0.018 radius=0.033; visual mesh filename=package://deepdrive_description/meshes/wheels/tire.stl scale=1 1 1
- added link tire_right_rear_link, mass 2.8498940e-02; collision cylinder length=0.018 radius=0.033; visual mesh filename=package://deepdrive_description/meshes/wheels/tire.stl scale=1 1 1
- added link wheel_left_rear_link, mass 2.8498940e-02; collision cylinder length=0.018 radius=0.033; visual mesh filename=package://deepdrive_description/meshes/wheels/rim.stl scale=1 1 1
- added link wheel_right_rear_link, mass 2.8498940e-02; collision cylinder length=0.018 radius=0.033; visual mesh filename=package://deepdrive_description/meshes/wheels/rim.stl scale=1 1 1
- link base_link: geometry collision box size=0.266 0.266 0.094; visual mesh filename=package://deepdrive_description/meshes/bases/deepdrive_chas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 scale=1 1 1
- link camera_link: geometry collision box size=0.012 0.132 0.020; visual mesh filename=package://deepdrive_description/meshes/sensors/oakdlite.stl
- link wheel_left_link: geometry collision cylinder length=0.018 radius=0.033; visual mesh filename=package://deepdrive_description/meshes/wheels/rim.stl scale=1 1 1
- link wheel_right_link: geometry collision cylinder length=0.018 radius=0.033; visual mesh filename=package://deepdrive_description/meshes/wheels/rim.stl scale=1 1 1
Joints:
- removed joint caster_back_left_joint
- removed joint caster_back_right_joint
- added joint tire_left_joint: type continuous, parent base_link, child tire_left_link, origin xyz=0.025 0.1 0.0 rpy=0 0 -1.57, axis 1 0 0
- added joint tire_left_rear_joint: type continuous, parent base_link, child tire_left_rear_link, origin xyz=-0.15 0.1 0.0 rpy=0 0 -1.57, axis 1 0 0
- added joint tire_right_joint: type continuous, parent base_link, child tire_right_link, origin xyz=0.025 -0.1 0.0 rpy=0 0 1.57, axis 1 0 0
- added joint tire_right_rear_joint: type continuous, parent base_link, child tire_right_rear_link, origin xyz=-0.15 -0.1 0.0 rpy=0 0 1.57, axis 1 0 0
- added joint wheel_left_rear_joint: type continuous, parent base_link, child wheel_left_rear_link, origin xyz=-0.15 0.1 0.0 rpy=0 0 -1.57, axis 1 0 0
- added joint wheel_right_rear_joint: type continuous, parent base_link, child wheel_right_rear_link, origin xyz=-0.15 -0.1 0.0 rpy=0 0 1.57, axis 1 0 0
- joint wheel_left_joint: axis 0 0 1 -> 1 0 0; origin xyz=0.0 0.144 0.023 rpy=-1.57 0 0 -> xyz=0.025 0.1 0.0 rpy=0 0 -1.57
- joint wheel_right_joint: axis 0 0 1 -> 1 0 0; origin xyz=0.0 -0.144 0.023 rpy=-1.57 0 0 -> xyz=0.025 -0.1 0.0 rpy=0 0 1.57

Commit message: Working on urdf

File: src/deepdrive_description/urdf/deepdrive_deepdrive.urdf (robot description, URDF)
Before this commit: robot deepdrive_deepdrive, 18 links, 17 joints
Links:
- removed link camera_depth_frame
- removed link camera_depth_optical_frame
- removed link camera_link
- removed link camera_rgb_frame
- removed link camera_rgb_optical_frame
- removed link imu_link
- removed link oak
Joints:
- removed joint camera_depth_joint
- removed joint camera_depth_optical_joint
- removed joint camera_joint
- removed joint camera_rgb_joint
- removed joint camera_rgb_optical_joint
- removed joint imu_joint
- removed joint oak_joint
- joint scan_joint: origin xyz=-0.064 0 0.122 rpy=0 0 0 -> xyz=-0.064 0 0.122 rpy=0 0 3.14

Commit message: rviz looking better

File: src/deepdrive_description/urdf/deepdrive_deepdrive.urdf (robot description, URDF)
Before this commit: robot deepdrive_deepdrive, 18 links, 17 joints
Links:
- removed link oak
- removed link tire_left_link
- removed link tire_left_rear_link
- removed link tire_right_link
- removed link tire_right_rear_link
- removed link wheel_left_link
- removed link wheel_left_rear_link
- removed link wheel_right_link
- removed link wheel_right_rear_link
- added link base_camera_link
- added link camera_wide_link; collision origin rpy=0 0 0 xyz=.017 .065 -.065; visual mesh filename=package://deepdrive_description/meshes/sensors/camera_wide.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 scale=.001 .001 .001
- added link laser
Joints:
- removed joint oak_joint
- removed joint tire_left_joint
- removed joint tire_left_rear_joint
- removed joint tire_right_joint
- removed joint tire_right_rear_joint
- removed joint wheel_left_joint
- removed joint wheel_left_rear_joint
- removed joint wheel_right_joint
- removed joint wheel_right_rear_joint
- added joint base_camera_joint: type fixed, parent base_link, child base_camera_link, origin xyz=0.0 0 0.068 rpy=0 0 1.57
- added joint camera_wide_joint: type fixed, parent base_link, child camera_wide_link, origin xyz=0.064 -0.065 0.094 rpy=0 0 0
- added joint laser_joint: type fixed, parent base_scan, child laser, origin xyz=0.0 0 0.068 rpy=0 0 1.57
- joint scan_joint: origin xyz=-0.064 0 0.122 rpy=0 0 0 -> xyz=-0.064 0 0.125 rpy=0 0 0

Commit message: working on urdf

File: src/deepdrive_description/urdf/deepdrive_deepdrive.urdf (robot description, URDF)
Before this commit: robot deepdrive_deepdrive, 11 links, 10 joints
Links:
- removed link base_camera_link
- removed link camera_depth_frame
- removed link camera_link
- removed link camera_rgb_frame
- removed link camera_rgb_optical_frame
- added link camera_depth
- added link camera_depth_depth_frame
- added link camera_depth_link, mass 0.061; collision box size=0.091 0.028 0.0175; visual mesh filename=package://deepdrive_description/meshes/sensors/oakdlite.stl
- added link camera_wide
- added link camera_wide_optical_frame
- added link tire_back_left_link, mass 2.8498940e-02; collision cylinder length=0.025 radius=0.035; visual mesh filename=package://deepdrive_description/meshes/wheels/tire.stl scale=1 1 1
- added link tire_back_right_link, mass 2.8498940e-02; collision cylinder length=0.025 radius=0.035; visual mesh filename=package://deepdrive_description/meshes/wheels/tire.stl scale=1 1 1
- added link tire_front_left_link, mass 2.8498940e-02; collision cylinder length=0.025 radius=0.035; visual mesh filename=package://deepdrive_description/meshes/wheels/tire.stl scale=1 1 1
- added link tire_front_right_link, mass 2.8498940e-02; collision cylinder length=0.025 radius=0.035; visual mesh filename=package://deepdrive_description/meshes/wheels/tire.stl scale=1 1 1
- added link wheel_back_left_link, mass 2.8498940e-02; collision cylinder length=0.025 radius=0.035; visual mesh filename=package://deepdrive_description/meshes/wheels/rim.stl scale=1 1 1
- added link wheel_back_right_link, mass 2.8498940e-02; collision cylinder length=0.025 radius=0.035; visual mesh filename=package://deepdrive_description/meshes/wheels/rim.stl scale=1 1 1
- added link wheel_front_left_link, mass 2.8498940e-02; collision cylinder length=0.025 radius=0.035; visual mesh filename=package://deepdrive_description/meshes/wheels/rim.stl scale=1 1 1
- added link wheel_front_right_link, mass 2.8498940e-02; collision cylinder length=0.025 radius=0.035; visual mesh filename=package://deepdrive_description/meshes/wheels/rim.stl scale=1 1 1
- link base_link: mass 1.3729096e+00 -> 2.3729096e+00; geometry collision box size=0.310 0.140 0.120; visual mesh filename=package://deepdrive_description/meshes/bases/deepdrive_chas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 scale=1 1 1
- link camera_wide_link: geometry collision box size=0.005 0.025 0.025; visual mesh filename=package://deepdrive_description/meshes/sensors/camera_wide.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 scale=.001 .001 .001
Joints:
- removed joint base_camera_joint
- removed joint camera_joint
- removed joint camera_rgb_joint
- removed joint camera_rgb_optical_joint
- added joint base_camera_depth_joint: type fixed, parent base_link, child camera_depth, origin xyz=0.08 0.0 0.035 rpy=0 0 0
- added joint base_camera_wide_joint: type fixed, parent base_link, child camera_wide, origin xyz=0.09 0.001 0.016 rpy=0 0 0
- added joint camera_depth_depth_joint: type fixed, parent camera_depth, child camera_depth_depth_frame, origin xyz=0 0 0 rpy=-1.5707963267948966 0 -1.5707963267948966
- added joint camera_wide_optical_joint: type fixed, parent camera_wide, child camera_wide_optical_frame, origin xyz=0 0 0 rpy=-1.5707963267948966 0 -1.5707963267948966
- added joint tire_back_left_joint: type fixed, parent wheel_back_left_link, child tire_back_left_link, origin xyz=0 0 0 rpy=0 0 0, axis 1 1 1
- added joint tire_back_right_joint: type fixed, parent wheel_back_right_link, child tire_back_right_link, origin xyz=0 0 0 rpy=0 0 0, axis 1 1 1
- added joint tire_front_left_joint: type fixed, parent wheel_front_left_link, child tire_front_left_link, origin xyz=0 0 0 rpy=0 0 0, axis 1 1 1
- added joint tire_front_right_joint: type fixed, parent wheel_front_right_link, child tire_front_right_link, origin xyz=0 0 0 rpy=0 0 0, axis 1 1 1
- added joint wheel_back_left_joint: type continuous, parent base_link, child wheel_back_left_link, origin xyz=0.022499999999999992 0.0875 0.0 rpy=0 0 -1.57, axis 1 0 0
- added joint wheel_back_right_joint: type continuous, parent base_link, child wheel_back_right_link, origin xyz=-0.1525 -0.0875 0.0 rpy=0 0 1.57, axis 1 0 0
- added joint wheel_front_left_joint: type continuous, parent base_link, child wheel_front_left_link, origin xyz=-0.1525 0.0875 0.0 rpy=0 0 -1.57, axis 1 0 0
- added joint wheel_front_right_joint: type continuous, parent base_link, child wheel_front_right_link, origin xyz=0.022499999999999992 -0.0875 0.0 rpy=0 0 1.57, axis 1 0 0
- joint camera_depth_joint: child camera_depth_frame -> camera_depth_link; origin xyz=0.005 0.028 0.013 rpy=0 0 0 -> xyz=0 0 0 rpy=0 0 0; parent camera_link -> camera_depth
- joint camera_depth_optical_joint: origin xyz=0 0 0 rpy=-1.57 0 -1.57 -> xyz=0 0 0 rpy=-1.5707963267948966 0 -1.5707963267948966; parent camera_depth_frame -> camera_depth
- joint camera_wide_joint: origin xyz=0.064 -0.065 0.094 rpy=0 0 0 -> xyz=0 0 0 rpy=0 0 0; parent base_link -> camera_wide
- joint laser_joint: origin xyz=0.0 0 0.068 rpy=0 0 1.57 -> xyz=0.0 0 0.058 rpy=0 0 1.57

Commit message: ros2_control hardware interface is working

File: src/deepdrive_description/urdf/deepdrive_deepdrive.urdf (robot description, URDF)
Before this commit: robot deepdrive_deepdrive, 19 links, 18 joints
Links:
- added link imu_link
- link tire_back_left_link: geometry visual mesh filename=package://deepdrive_description/meshes/wheels/tire.stl scale=1 1 1
- link tire_back_right_link: geometry visual mesh filename=package://deepdrive_description/meshes/wheels/tire.stl scale=1 1 1
- link tire_front_left_link: geometry visual mesh filename=package://deepdrive_description/meshes/wheels/tire.stl scale=1 1 1
- link tire_front_right_link: geometry visual mesh filename=package://deepdrive_description/meshes/wheels/tire.stl scale=1 1 1
- link wheel_back_left_link: mass 2.8498940e-02 -> .05
- link wheel_back_right_link: mass 2.8498940e-02 -> .05
- link wheel_front_left_link: mass 2.8498940e-02 -> .05
- link wheel_front_right_link: mass 2.8498940e-02 -> .05
Joints:
- added joint imu_joint: type fixed, parent base_link, child imu_link, origin xyz=0.0 0 0.068 rpy=0 0 0
- joint wheel_back_left_joint: axis 1 0 0 -> -1 0 0; origin xyz=0.022499999999999992 0.0875 0.0 rpy=0 0 -1.57 -> xyz=-0.1525 0.0875 0.0 rpy=0 0 -1.57
- joint wheel_front_left_joint: axis 1 0 0 -> -1 0 0; origin xyz=-0.1525 0.0875 0.0 rpy=0 0 -1.57 -> xyz=0.022499999999999992 0.0875 0.0 rpy=0 0 -1.57

File: src/deepdrive_description/urdf/deepdrive_deepdrive.xacro (robot description, xacro)
@@ -2,6 +2,8 @@
 <robot name="deepdrive_deepdrive"
   xmlns:xacro="http://ros.org/wiki/xacro">
+  <xacro:arg name="sim_mode" default="false"/>
   <xacro:property name="wheel_base" value="0.175" />
   <xacro:property name="wheel_radius" value="0.035" />
+  <!-- <xacro:property name="use_mock_hardware" value="0.035" /> -->
   <xacro:include filename="$(find deepdrive_description)/urdf/common_properties.xacro"/>
   <xacro:include filename="$(find deepdrive_description)/urdf/wheels.xacro"/>
@@ -55,77 +57,49 @@
   <xacro:include filename="$(find deepdrive_description)/urdf/lidar.xacro" />
   <xacro:include filename="$(find deepdrive_description)/urdf/camera.xacro" />
-  <ros2_control name="GazeboSystem" type="system">
-    <hardware>
-      <plugin>gazebo_ros2_control/GazeboSystem</plugin>
-    </hardware>
-  <!-- <hardware>
-      <plugin>mock_components/GenericSystem</plugin>
-      <param name="calculate_dynamics">true</param>
-    </hardware> -->
-  <joint name="wheel_front_left_joint">
+  <!-- ros2_control -->
+  <xacro:macro name="ros2_wheel_joint" params="name">
+    <joint name="wheel_${name}_joint">
       <command_interface name="velocity">
-        <param name="min">-10</param>
-        <param name="max">10</param>
+        <param name="min">-1</param>
+        <param name="max">1</param>
       </command_interface>
       <state_interface name="position" />
       <state_interface name="velocity" />
     </joint>
-    <joint name="wheel_front_right_joint">
-      <command_interface name="velocity">
-        <param name="min">-10</param>
-        <param name="max">10</param>
-      </command_interface>
-      <state_interface name="velocity" />
-      <state_interface name="position" />
-    </joint>
-    <joint name="wheel_back_left_joint">
-      <command_interface name="velocity">
-        <param name="min">-10</param>
-        <param name="max">10</param>
-      </command_interface>
-      <state_interface name="position" />
-      <state_interface name="velocity" />
-    </joint>
-    <joint name="wheel_back_right_joint">
-      <command_interface name="velocity">
-        <param name="min">-10</param>
-        <param name="max">10</param>
-      </command_interface>
-      <state_interface name="velocity" />
-      <state_interface name="position" />
-    </joint>
-  </ros2_control>
-  <!-- <ros2_control name="${name}" type="system">
-    <xacro:unless value="${use_mock_hardware}">
+  </xacro:macro>
+  <ros2_control name="GazeboSystem" type="system">
+    <!-- Gazebo simulation -->
+    <xacro:if value="$(arg sim_mode)">
       <hardware>
-        <plugin>ros2_control_demo_example_2/DiffBotSystemHardware</plugin>
-        <param name="example_param_hw_start_duration_sec">0</param>
-        <param name="example_param_hw_stop_duration_sec">3.0</param>
+        <plugin>gazebo_ros2_control/GazeboSystem</plugin>
+      </hardware>
+    </xacro:if>
+    <!-- Physical Robot -->
+    <xacro:unless value="$(arg sim_mode)">
+      <hardware>
+        <plugin>deepdrive_control/DeepdriveSystemHardware</plugin>
+        <param name="mock_hardware">true</param>
+        <param name="pin_left_enable">32</param>
+        <param name="pin_left_forward">38</param>
+        <param name="pin_left_backward">37</param>
+        <param name="pin_right_enable">33</param>
+        <param name="pin_right_forward">35</param>
+        <param name="pin_right_backward">36</param>
+        <param name="pwm_hz">50</param>
       </hardware>
     </xacro:unless>
-    <xacro:if value="${use_mock_hardware}">
-      <hardware>
-        <plugin>mock_components/GenericSystem</plugin>
-        <param name="calculate_dynamics">true</param>
-      </hardware>
-    </xacro:if>
-    <joint name="${prefix}left_wheel_joint">
-      <command_interface name="velocity"/>
-      <state_interface name="position"/>
-      <state_interface name="velocity"/>
-    </joint>
-    <joint name="${prefix}right_wheel_joint">
-      <command_interface name="velocity"/>
-      <state_interface name="position"/>
-      <state_interface name="velocity"/>
-    </joint>
-  </ros2_control> -->
-  <gazebo>
-    <plugin filename="libgazebo_ros2_control.so" name="gazebo_ros2_control">
-      <parameters>$(find deepdrive_description)/config/controllers.yaml</parameters>
-    </plugin>
-  </gazebo>
-<!-- This one works in gazebo -->
-  <!-- <gazebo>
+    <xacro:ros2_wheel_joint name="back_right" />
+    <xacro:ros2_wheel_joint name="front_left" />
+    <xacro:ros2_wheel_joint name="back_left" />
+    <xacro:ros2_wheel_joint name="front_right" />
+  </ros2_control>
+  <xacro:if value="$(arg sim_mode)">
+    <gazebo>
+      <plugin filename="libgazebo_ros2_control.so" name="gazebo_ros2_control">
+        <parameters>$(find deepdrive_description)/config/controllers.yaml</parameters>
+      </plugin>
+    </gazebo>
+    <!-- This one works in gazebo without ros2_control -->
+    <!-- <gazebo>
     <plugin name='diff_drive' filename='libgazebo_ros_diff_drive.so'>
       <num_wheel_pairs>2</num_wheel_pairs>
@@ -145,71 +119,72 @@
     </plugin>
   </gazebo> -->
-  <gazebo reference="imu_link">
-    <sensor name="imu_sensor" type="imu">
-      <plugin filename="libgazebo_ros_imu_sensor.so" name="imu_plugin">
-        <ros>
-          <namespace>/</namespace>
-          <remapping>~/out:=imu</remapping>
-        </ros>
-        <initial_orientation_as_reference>false</initial_orientation_as_reference>
-      </plugin>
-      <always_on>true</always_on>
-      <update_rate>100</update_rate>
-      <visualize>true</visualize>
-      <imu>
-        <angular_velocity>
-          <x>
-            <noise type="gaussian">
-              <mean>0.0</mean>
-              <stddev>2e-4</stddev>
-              <bias_mean>0.0000075</bias_mean>
-              <bias_stddev>0.0000008</bias_stddev>
-            </noise>
-          </x>
-          <y>
-            <noise type="gaussian">
-              <mean>0.0</mean>
-              <stddev>2e-4</stddev>
-              <bias_mean>0.0000075</bias_mean>
-              <bias_stddev>0.0000008</bias_stddev>
-            </noise>
-          </y>
-          <z>
-            <noise type="gaussian">
-              <mean>0.0</mean>
-              <stddev>2e-4</stddev>
-              <bias_mean>0.0000075</bias_mean>
-              <bias_stddev>0.0000008</bias_stddev>
-            </noise>
-          </z>
-        </angular_velocity>
-        <linear_acceleration>
-          <x>
-            <noise type="gaussian">
-              <mean>0.0</mean>
-              <stddev>1.7e-2</stddev>
-              <bias_mean>0.1</bias_mean>
-              <bias_stddev>0.001</bias_stddev>
-            </noise>
-          </x>
-          <y>
-            <noise type="gaussian">
-              <mean>0.0</mean>
-              <stddev>1.7e-2</stddev>
-              <bias_mean>0.1</bias_mean>
-              <bias_stddev>0.001</bias_stddev>
-            </noise>
-          </y>
-          <z>
-            <noise type="gaussian">
-              <mean>0.0</mean>
-              <stddev>1.7e-2</stddev>
-              <bias_mean>0.1</bias_mean>
-              <bias_stddev>0.001</bias_stddev>
-            </noise>
-          </z>
-        </linear_acceleration>
-      </imu>
-    </sensor>
-  </gazebo>
+    <gazebo reference="imu_link">
+      <sensor name="imu_sensor" type="imu">
+        <plugin filename="libgazebo_ros_imu_sensor.so" name="imu_plugin">
+          <ros>
+            <namespace>/</namespace>
+            <remapping>~/out:=imu</remapping>
+          </ros>
+          <initial_orientation_as_reference>false</initial_orientation_as_reference>
+        </plugin>
+        <always_on>true</always_on>
+        <update_rate>100</update_rate>
+        <visualize>true</visualize>
+        <imu>
+          <angular_velocity>
+            <x>
+              <noise type="gaussian">
+                <mean>0.0</mean>
+                <stddev>2e-4</stddev>
+                <bias_mean>0.0000075</bias_mean>
+                <bias_stddev>0.0000008</bias_stddev>
+              </noise>
+            </x>
+            <y>
+              <noise type="gaussian">
+                <mean>0.0</mean>
+                <stddev>2e-4</stddev>
+                <bias_mean>0.0000075</bias_mean>
+                <bias_stddev>0.0000008</bias_stddev>
+              </noise>
+            </y>
+            <z>
+              <noise type="gaussian">
+                <mean>0.0</mean>
+                <stddev>2e-4</stddev>
+                <bias_mean>0.0000075</bias_mean>
+                <bias_stddev>0.0000008</bias_stddev>
+              </noise>
+            </z>
+          </angular_velocity>
+          <linear_acceleration>
+            <x>
+              <noise type="gaussian">
+                <mean>0.0</mean>
+                <stddev>1.7e-2</stddev>
+                <bias_mean>0.1</bias_mean>
+                <bias_stddev>0.001</bias_stddev>
+              </noise>
+            </x>
+            <y>
+              <noise type="gaussian">
+                <mean>0.0</mean>
+                <stddev>1.7e-2</stddev>
+                <bias_mean>0.1</bias_mean>
+                <bias_stddev>0.001</bias_stddev>
+              </noise>
+            </y>
+            <z>
+              <noise type="gaussian">
+                <mean>0.0</mean>
+                <stddev>1.7e-2</stddev>
+                <bias_mean>0.1</bias_mean>
+                <bias_stddev>0.001</bias_stddev>
+              </noise>
+            </z>
+          </linear_acceleration>
+        </imu>
+      </sensor>
+    </gazebo>
+  </xacro:if>
 </robot>

File: src/deepdrive_description/urdf/ros2_control.xacro (robot description, xacro)
@@ -56,5 +56,5 @@
     <gazebo>
         <plugin name="gazebo_ros2_control" filename="libgazebo_ros2_control.so">
-            <parameters>$(find deepdrive_description)/config/controllers.yaml</parameters>
+            <parameters>$(find deepdrive_description)/config/controllers_sim.yaml</parameters>
             <parameters>$(find deepdrive_description)/config/gaz_ros2_ctl_use_sim.yaml</parameters>
         </plugin>
