Commit message: Working on nav2

File: src/deepdrive_description/urdf/deepdrive_deepdrive.urdf (robot description, URDF)
Before this commit: robot deepdrive_deepdrive, 20 links, 19 joints
Joints:
- joint camera_depth_optical_joint: origin xyz=0 0 0 rpy=-1.5707963267948966 0 -1.5707963267948966 -> xyz=0.1 0 0.2 rpy=-1.5707963267948966 0 -1.5707963267948966
- joint laser_joint: origin xyz=0.0 0 0.058 rpy=0 0 1.57 -> xyz=0.0 0 0.058 rpy=0 0 3.141592653589793
