Commit message: Working on bringup and odom

File: src/deepdrive_description/urdf/camera.xacro (robot description, xacro)
@@ -6,5 +6,5 @@
         <parent link="base_link"/>
         <child link="camera_depth"/>
-        <origin xyz="0.08 0.0 0.035" rpy="0 0 0"/>
+        <origin xyz="0.14 -0.045 0.09" rpy="0 0 0"/>
     </joint>
     <link name="camera_depth"/>
@@ -15,5 +15,6 @@
         <parent link="base_link"/>
         <child link="camera_wide"/>
-        <origin xyz="0.09 0.001 0.016" rpy="0 0 0"/>
+        <origin xyz="0.125 0.030 0.081" rpy="0 0 0"/>
+        <!-- <origin xyz="0.125 0.03 0.08" rpy="${-pi/2} 0 ${-pi/2}"/> -->
         <!-- <origin xyz="0.064 -0.065 0.094" rpy="0 0 0"/> -->
         <!-- 0 1.57 0 -->
@@ -22,49 +23,3 @@
     <link name="camera_wide"/>
     <xacro:camera_wide mount_point="camera_wide"/>
-    <!-- <joint name="camera_joint" type="fixed">
-        <origin xyz="0.064 -0.065 0.094" rpy="0 0 0"/>
-        <parent link="base_link"/>
-        <child link="camera_link"/>
-    </joint> -->
-<!--
-    <link name="camera_link">
-        <visual>
-            <origin xyz=".01 .065 -.025" rpy="1.57 0 1.57"/>
-            <geometry>
-                <mesh filename="package://deepdrive_description/meshes/sensors/oakdlite.stl" />
-            </geometry>
-            <material name="black"/>
-        </visual>
-        <collision>
-            <origin xyz="0.003 0.065 0.007" rpy="0 0 0"/>
-            <geometry>
-                <box size="0.012 0.132 0.020"/>
-            </geometry>
-        </collision>
-    </link>
-    <joint name="camera_rgb_joint" type="fixed">
-        <origin xyz="0.005 0.018 0.013" rpy="0 0 0"/>
-        <parent link="camera_link"/>
-        <child link="camera_rgb_frame"/>
-    </joint>
-    <link name="camera_rgb_frame"/>
-    <joint name="camera_rgb_optical_joint" type="fixed">
-        <origin xyz="0 0 0" rpy="-1.57 0 -1.57"/>
-        <parent link="camera_rgb_frame"/>
-        <child link="camera_rgb_optical_frame"/>
-    </joint>
-    <link name="camera_rgb_optical_frame"/>
-    <joint name="camera_depth_joint" type="fixed">
-        <origin xyz="0.005 0.028 0.013" rpy="0 0 0"/>
-        <parent link="camera_link"/>
-        <child link="camera_depth_frame"/>
-    </joint>
-    <link name="camera_depth_frame"/>
-    <joint name="camera_depth_optical_joint" type="fixed">
-        <origin xyz="0 0 0" rpy="-1.57 0 -1.57"/>
-        <parent link="camera_depth_frame"/>
-        <child link="camera_depth_optical_frame"/>
-    </joint>
-    <link name="camera_depth_optical_frame"/> -->
-    <!-- Gazebo plugin for center RGB camera -->
 </robot>

File: src/deepdrive_description/urdf/camera_wide.xacro (robot description, xacro)
@@ -4,5 +4,5 @@
         <!-- Wide angle camera -->
         <joint name="${mount_point}_joint" type="fixed">
-            <origin xyz="0 0 0" rpy="0 0 0"/>
+            <origin xyz="0 0 0" rpy="${-pi/2} 0 ${-pi/2}"/>
             <parent link="${mount_point}"/>
             <child link="${mount_point}_link"/>
@@ -10,5 +10,5 @@
         <link name="${mount_point}_link">
             <visual>
-                <origin xyz="-0.01 -0.015 0.001" rpy="${pi/2} 0 ${pi/2}"/>
+                <origin xyz="0 0 0" rpy="0 0 ${pi/2}"/>
                 <geometry>
                     <mesh filename="package://deepdrive_description/meshes/sensors/camera_wide.stl" scale=".001 .001 .001"/>
@@ -24,5 +24,6 @@
         </link>
         <joint name="${mount_point}_optical_joint" type="fixed">
-            <origin xyz="0 0 0" rpy="${-pi/2} 0 ${-pi/2}"/>
+            <origin xyz="0 0 0" rpy="0 0 0"/>
+            <!-- <origin xyz="0 0 0" rpy="${-pi/2} 0 ${-pi/2}"/> -->
             <parent link="${mount_point}"/>
             <child link="${mount_point}_optical_frame"/>

File: src/deepdrive_description/urdf/common_properties.xacro (robot description, xacro)
@@ -21,4 +21,7 @@
     <color rgba="0.5 0.5 0.5 1.0"/>
   </material>
+  <material name="lightgrey">
+    <color rgba="0.7 0.7 0.7 1.0"/>
+  </material>
   <material name="orange">
     <color rgba="${255/255} ${108/255} ${10/255} 1.0"/>

File: src/deepdrive_description/urdf/deepdrive_deepdrive.urdf (robot description, URDF)
Before this commit: robot deepdrive_deepdrive, 20 links, 19 joints
Links:
- removed link base_scan
- removed link laser
- added link body_link; visual mesh filename=package://deepdrive_description/meshes/bases/body.stl scale=.001 .001 .001
- added link camera_depth_imu_frame
- added link camera_depth_left_camera_optical_frame
- added link camera_depth_rgb_camera_optical_frame
- added link camera_depth_right_camera_optical_frame
- added link ldlidar_base; visual mesh filename=package://ldlidar_node/urdf/model/LD19.stl scale=0.001 0.001 0.001
- added link ldlidar_link
- link base_link: geometry collision box size=0.310 0.140 0.120; visual mesh filename=package://deepdrive_description/meshes/bases/chassis.stl scale=.001 .001 .001
- link tire_back_left_link: geometry visual mesh filename=package://deepdrive_description/meshes/wheels/tire.stl scale=.001 .001 .001
- link tire_back_right_link: geometry visual mesh filename=package://deepdrive_description/meshes/wheels/tire.stl scale=.001 .001 .001
- link tire_front_left_link: geometry visual mesh filename=package://deepdrive_description/meshes/wheels/tire.stl scale=.001 .001 .001
- link tire_front_right_link: geometry visual mesh filename=package://deepdrive_description/meshes/wheels/tire.stl scale=.001 .001 .001
- link wheel_back_left_link: geometry collision cylinder length=0.025 radius=0.0445; visual mesh filename=package://deepdrive_description/meshes/wheels/rim.stl scale=.001 .001 .001
- link wheel_back_right_link: geometry collision cylinder length=0.025 radius=0.0445; visual mesh filename=package://deepdrive_description/meshes/wheels/rim.stl scale=.001 .001 .001
- link wheel_front_left_link: geometry collision cylinder length=0.025 radius=0.0445; visual mesh filename=package://deepdrive_description/meshes/wheels/rim.stl scale=.001 .001 .001
- link wheel_front_right_link: geometry collision cylinder length=0.025 radius=0.0445; visual mesh filename=package://deepdrive_description/meshes/wheels/rim.stl scale=.001 .001 .001
Joints:
- removed joint laser_joint
- removed joint scan_joint
- added joint body_joint: type fixed, parent base_link, child body_link, origin xyz=0 0 0.0 rpy=0 0 0
- added joint camera_depth_imu_link: type fixed, parent camera_depth_link, child camera_depth_imu_frame, origin xyz=0.0 0 0.0 rpy=-1.5707963267948966 0 1.5707963267948966
- added joint camera_depth_left_camera_optical_frame_joint: type fixed, parent camera_depth_optical_frame, child camera_depth_left_camera_optical_frame, origin xyz=0 0 0 rpy=0 0 0
- added joint camera_depth_rgb_camera_optical_frame_joint: type fixed, parent camera_depth_optical_frame, child camera_depth_rgb_camera_optical_frame, origin xyz=0 0 0 rpy=0 0 0
- added joint camera_depth_right_camera_optical_frame_joint: type fixed, parent camera_depth_optical_frame, child camera_depth_right_camera_optical_frame, origin xyz=0 0 0 rpy=0 0 0
- added joint ldlidar_joint: type fixed, parent base_link, child ldlidar_base, origin xyz=-0.05 0.001 0.120 rpy=0 0 0
- added joint ldlidar_link_joint: type fixed, parent ldlidar_base, child ldlidar_link, origin xyz=0 0 0 rpy=0 0 0
- joint base_camera_depth_joint: origin xyz=0.08 0.0 0.035 rpy=0 0 0 -> xyz=0.14 -0.045 0.09 rpy=0 0 0
- joint base_camera_wide_joint: origin xyz=0.09 0.001 0.016 rpy=0 0 0 -> xyz=0.125 0.030 0.081 rpy=0 0 0
- joint camera_depth_depth_joint: origin xyz=0 0 0 rpy=-1.5707963267948966 0 -1.5707963267948966 -> xyz=0 0 0 rpy=0 0 0
- joint camera_depth_optical_joint: origin xyz=0.1 0 0.2 rpy=-1.5707963267948966 0 -1.5707963267948966 -> xyz=0 0 0 rpy=-1.5707963267948966 0 -1.5707963267948966
- joint camera_wide_optical_joint: origin xyz=0 0 0 rpy=-1.5707963267948966 0 -1.5707963267948966 -> xyz=0 0 0 rpy=0 0 0
- joint wheel_back_left_joint: origin xyz=-0.1525 0.0875 0.0 rpy=0 0 -1.57 -> xyz=-0.185 0.12 0.0 rpy=0 0 -1.5707963267948966
- joint wheel_back_right_joint: origin xyz=-0.1525 -0.0875 0.0 rpy=0 0 1.57 -> xyz=-0.185 -0.12 0.0 rpy=0 0 1.5707963267948966
- joint wheel_front_left_joint: origin xyz=0.022499999999999992 0.0875 0.0 rpy=0 0 -1.57 -> xyz=0.05499999999999999 0.12 0.0 rpy=0 0 -1.5707963267948966
- joint wheel_front_right_joint: origin xyz=0.022499999999999992 -0.0875 0.0 rpy=0 0 1.57 -> xyz=0.05499999999999999 -0.12 0.0 rpy=0 0 1.5707963267948966

File: src/deepdrive_description/urdf/deepdrive_deepdrive.xacro (robot description, xacro)
@@ -3,6 +3,6 @@
   xmlns:xacro="http://ros.org/wiki/xacro">
   <xacro:arg name="sim_mode" default="false"/>
-  <xacro:property name="wheel_base" value="0.175" />
-  <xacro:property name="wheel_radius" value="0.035" />
+  <xacro:property name="wheel_base" value="0.24" />
+  <xacro:property name="wheel_radius" value="0.0445" />
   <!-- <xacro:property name="use_mock_hardware" value="true" /> -->
   <xacro:include filename="$(find deepdrive_description)/urdf/common_properties.xacro"/>
@@ -14,11 +14,12 @@
     <origin xyz="0 0 0.010" rpy="0 0 0"/>
   </joint>
+  <!-- Frame/Chassis -->
   <link name="base_link">
     <visual>
-      <origin xyz="-0.064 0 0.0" rpy="0 0 1.57"/>
+      <origin xyz="-0.064 0 0.0" rpy="0 0 ${pi/2}"/>
       <geometry>
-        <mesh filename="package://deepdrive_description/meshes/bases/deepdrive_chassis.stl" scale="1 1 1"/>
+        <mesh filename="package://deepdrive_description/meshes/bases/chassis.stl" scale=".001 .001 .001"/>
       </geometry>
-      <material name="grey"/>
+      <material name="dark"/>
     </visual>
     <collision>
@@ -37,8 +38,28 @@
     <material>Gazebo/Grey</material>
   </gazebo>
+  <!-- Body-->
+  <joint name="body_joint" type="fixed">
+    <parent link="base_link"/>
+    <child link="body_link" />
+    <origin xyz="0 0 0.0" rpy="0 0 0"/>
+  </joint>
+  <link name="body_link">
+    <visual>
+      <origin xyz="-0.064 0 0.0" rpy="0 0 ${pi/2}"/>
+      <geometry>
+        <mesh filename="package://deepdrive_description/meshes/bases/body.stl" scale=".001 .001 .001"/>
+      </geometry>
+      <material name="black"/>
+    </visual>
+  </link>
+  <gazebo reference="base_link">
+    <material>Gazebo/Black</material>
+  </gazebo>
+  <!-- Wheels -->
   <xacro:wheel name="front_right" lr="1" fb="1" wheel_base="${wheel_base}" wheel_radius="${wheel_radius}" />
   <xacro:wheel name="back_right" lr="1" fb="-1" wheel_base="${wheel_base}" wheel_radius="${wheel_radius}" />
   <xacro:wheel name="front_left" lr="-1" fb="1" wheel_base="${wheel_base}" wheel_radius="${wheel_radius}" />
   <xacro:wheel name="back_left" lr="-1" fb="-1" wheel_base="${wheel_base}" wheel_radius="${wheel_radius}" />
+  <!-- IMU -->
   <joint name="imu_joint" type="fixed">
     <parent link="base_link"/>
@@ -47,11 +68,11 @@
   </joint>
   <link name="imu_link"/>
-   <!-- <joint name="oak_joint" type="fixed">
+  <!-- LIDAR -->
+  <joint name="ldlidar_joint" type="fixed">
     <parent link="base_link"/>
-    <child link="camera_depth_imu_frame"/>
-    <origin xyz="0.0 0 0.0" rpy="0 0 0"/>
-  </joint> -->
-  <!-- <link name="camera_depth_imu_frame"/> -->
-  <!-- LIDAR -->
+    <child link="ldlidar_base"/>
+    <origin xyz="-0.05 0.001 0.120" rpy="0 0 0"/>
+  </joint>
+  <!-- <link name="imu_link"/> -->
   <xacro:include filename="$(find deepdrive_description)/urdf/lidar.xacro" />
   <xacro:include filename="$(find deepdrive_description)/urdf/camera.xacro" />

File: src/deepdrive_description/urdf/lidar.xacro (robot description, xacro)
@@ -15,5 +15,5 @@
         <parent link="ldlidar_base"/>
         <child link="ldlidar_link"/>
-        <origin xyz="0 0 0.02745" rpy="0 0 0" />
+        <origin xyz="0 0 0" rpy="0 0 0" />
     </joint>
     <link name="ldlidar_link" />

File: src/deepdrive_description/urdf/oakdlite.xacro (robot description, xacro)
@@ -15,5 +15,5 @@
     <link name="${mount_point}_link">
       <visual>
-        <origin xyz="-0.01 0.00 0.030" rpy="${pi/2} 0 ${pi/2}"/>
+        <origin xyz="0 0 0" rpy="${pi/2} 0 ${pi/2}"/>
         <geometry>
           <mesh filename="package://deepdrive_description/meshes/sensors/oakdlite.stl" />
@@ -29,11 +29,18 @@
       <xacro:solid_cuboid_inertial rpy="0 0 0" xyz="0 0 0" mass="${oakd_mass}" x="${oakd_length}" y="${oakd_width}" z="${oakd_depth}" />
     </link>
+    <joint name="${mount_point}_imu_link" type="fixed">
+      <parent link="${mount_point}_link"/>
+      <child link="${mount_point}_imu_frame"/>
+      <origin xyz="0.0 0 0.0" rpy="${-pi/2} 0 ${pi/2}"/>
+    </joint>
+    <link name="${mount_point}_imu_frame"/>
     <!-- RGB -->
     <joint name="${mount_point}_optical_joint" type="fixed">
-      <origin xyz="0.1 0 0.2" rpy="${-pi/2} 0 ${-pi/2}"/>
+      <origin xyz="0 0 0" rpy="${-pi/2} 0 ${-pi/2}"/>
       <parent link="${mount_point}"/>
       <child link="${mount_point}_optical_frame"/>
     </joint>
     <link name="${mount_point}_optical_frame"/>
+    <!-- Gazebo -->
     <sensor type="camera" name="${mount_point}_rgb">
       <!-- Seems to be ignored -->
@@ -65,9 +72,29 @@
     <!-- Depth/Stereo -->
     <joint name="${mount_point}_depth_joint" type="fixed">
-      <origin xyz="0 0 0" rpy="${-pi/2} 0 ${-pi/2}"/>
+      <origin xyz="0 0 0" rpy="0 0 0"/>
       <parent link="${mount_point}"/>
       <child link="${mount_point}_depth_frame"/>
     </joint>
     <link name="${mount_point}_depth_frame"/>
+    <!-- TODO: Not sure why these are popping up in foxglove, but just hack them for now -->
+    <joint name="${mount_point}_right_camera_optical_frame_joint" type="fixed">
+      <origin xyz="0 0 0" rpy="0 0 0"/>
+      <parent link="${mount_point}_optical_frame"/>
+      <child link="${mount_point}_right_camera_optical_frame"/>
+    </joint>
+    <link name="${mount_point}_right_camera_optical_frame"/>
+    <joint name="${mount_point}_left_camera_optical_frame_joint" type="fixed">
+      <origin xyz="0 0 0" rpy="0 0 0"/>
+      <parent link="${mount_point}_optical_frame"/>
+      <child link="${mount_point}_left_camera_optical_frame"/>
+    </joint>
+    <link name="${mount_point}_left_camera_optical_frame"/>
+    <joint name="${mount_point}_rgb_camera_optical_frame_joint" type="fixed">
+      <origin xyz="0 0 0" rpy="0 0 0"/>
+      <parent link="${mount_point}_optical_frame"/>
+      <child link="${mount_point}_rgb_camera_optical_frame"/>
+    </joint>
+    <link name="${mount_point}_rgb_camera_optical_frame"/>
+    <!-- end hack -->
     <gazebo reference="${mount_point}_link">
       <material>Gazebo/Black</material>

File: src/deepdrive_description/urdf/wheels.xacro (robot description, xacro)
@@ -8,5 +8,5 @@
             <parent link="base_link"/>
             <child link="wheel_${name}_link"/>
-            <origin xyz="${wheel_front_offset/2 + (fb * (wheel_base / 2))} ${-lr * wheel_base/2} 0.0" rpy="0 0 ${lr*1.57}"/>
+        <origin xyz="${wheel_front_offset/2 + (fb * (wheel_base / 2))} ${-lr * wheel_base/2} 0.0" rpy="0 0 ${lr*(pi/2)}"/>
             <axis xyz="${lr} 0 0"/>
             <!-- <dynamics damping="0.8"/> -->
@@ -25,7 +25,7 @@
                 <origin xyz="0 0 0" rpy="0 0 0"/>
                 <geometry>
-                    <mesh filename="package://deepdrive_description/meshes/wheels/rim.stl" scale="1 1 1"/>
+                    <mesh filename="package://deepdrive_description/meshes/wheels/rim.stl" scale=".001 .001 .001"/>
                 </geometry>
-                <material name="blue"/>
+                <material name="dark"/>
             </visual>
             <collision>
@@ -42,5 +42,5 @@
         </link>
         <gazebo reference="wheel_${name}_link">
-            <material>Gazebo/Blue</material>
+            <material>Gazebo/Grey</material>
         </gazebo>
         <joint name="tire_${name}_joint" type="fixed">
@@ -54,5 +54,5 @@
                 <origin xyz="0 0 0" rpy="0 0 0"/>
                 <geometry>
-                    <mesh filename="package://deepdrive_description/meshes/wheels/tire.stl" scale="1 1 1"/>
+                    <mesh filename="package://deepdrive_description/meshes/wheels/tire.stl" scale=".001 .001 .001"/>
                 </geometry>
                 <material name="black"/>
