Commit message: simulator working with skid steer, imu and joystick

File: src/deepdrive_description/urdf/deepdrive_deepdrive.xacro (robot description, xacro)
@@ -37,7 +37,7 @@
   <xacro:wheel name="front_right" lr="1" fb="1" wheel_base="${wheel_base}" wheel_radius="${wheel_radius}" />
   <xacro:wheel name="back_right" lr="1" fb="-1" wheel_base="${wheel_base}" wheel_radius="${wheel_radius}" />
-  <xacro:wheel name="front_left" lr="-1" fb="-1" wheel_base="${wheel_base}" wheel_radius="${wheel_radius}" />
-  <xacro:wheel name="back_left" lr="-1" fb="1" wheel_base="${wheel_base}" wheel_radius="${wheel_radius}" />
-  <!-- <joint name="imu_joint" type="fixed">
+  <xacro:wheel name="front_left" lr="-1" fb="1" wheel_base="${wheel_base}" wheel_radius="${wheel_radius}" />
+  <xacro:wheel name="back_left" lr="-1" fb="-1" wheel_base="${wheel_base}" wheel_radius="${wheel_radius}" />
+  <joint name="imu_joint" type="fixed">
     <parent link="base_link"/>
     <child link="imu_link"/>
@@ -45,4 +45,5 @@
   </joint>
   <link name="imu_link"/>
+  <!--
    <joint name="oak_joint" type="fixed">
     <parent link="base_link"/>
@@ -54,4 +55,168 @@
   <xacro:include filename="$(find deepdrive_description)/urdf/lidar.xacro" />
   <xacro:include filename="$(find deepdrive_description)/urdf/camera.xacro" />
+  <!-- <ros2_control name="GazeboSystem" type="system">
+    <hardware>
+      <plugin>gazebo_ros2_control/GazeboSystem</plugin>
+    </hardware> -->
+  <!-- <hardware>
+      <plugin>mock_components/GenericSystem</plugin>
+      <param name="calculate_dynamics">true</param>
+    </hardware> -->
+  <!-- <joint name="wheel_front_left_joint">
+      <command_interface name="velocity">
+        <param name="min">-10</param>
+        <param name="max">10</param>
+      </command_interface>
+      <state_interface name="position" />
+      <state_interface name="velocity" />
+    </joint>
+    <joint name="wheel_front_right_joint">
+      <command_interface name="velocity">
+        <param name="min">-10</param>
+        <param name="max">10</param>
+      </command_interface>
+      <state_interface name="velocity" />
+      <state_interface name="position" />
+    </joint>
+    <joint name="wheel_back_left_joint">
+      <command_interface name="velocity">
+        <param name="min">-10</param>
+        <param name="max">10</param>
+      </command_interface>
+      <state_interface name="position" />
+      <state_interface name="velocity" />
+    </joint>
+    <joint name="wheel_back_right_joint">
+      <command_interface name="velocity">
+        <param name="min">-10</param>
+        <param name="max">10</param>
+      </command_interface>
+      <state_interface name="velocity" />
+      <state_interface name="position" />
+    </joint>
+  </ros2_control> -->
+  <!-- <ros2_control name="${name}" type="system">
+    <xacro:unless value="${use_mock_hardware}">
+      <hardware>
+        <plugin>ros2_control_demo_example_2/DiffBotSystemHardware</plugin>
+        <param name="example_param_hw_start_duration_sec">0</param>
+        <param name="example_param_hw_stop_duration_sec">3.0</param>
+      </hardware>
+    </xacro:unless>
+    <xacro:if value="${use_mock_hardware}">
+      <hardware>
+        <plugin>mock_components/GenericSystem</plugin>
+        <param name="calculate_dynamics">true</param>
+      </hardware>
+    </xacro:if>
+    <joint name="${prefix}left_wheel_joint">
+      <command_interface name="velocity"/>
+      <state_interface name="position"/>
+      <state_interface name="velocity"/>
+    </joint>
+    <joint name="${prefix}right_wheel_joint">
+      <command_interface name="velocity"/>
+      <state_interface name="position"/>
+      <state_interface name="velocity"/>
+    </joint>
+  </ros2_control> -->
+  <!-- <gazebo>
+    <plugin filename="libgazebo_ros2_control.so" name="gazebo_ros2_control">
+      <parameters>$(find deepdrive_description)/config/controllers.yaml</parameters>
+    </plugin>
+  </gazebo> -->
+  <gazebo reference="imu_link">
+    <sensor name="imu_sensor" type="imu">
+      <plugin filename="libgazebo_ros_imu_sensor.so" name="imu_plugin">
+        <ros>
+          <namespace>/</namespace>
+          <remapping>~/out:=imu</remapping>
+        </ros>
+        <initial_orientation_as_reference>false</initial_orientation_as_reference>
+      </plugin>
+      <always_on>true</always_on>
+      <update_rate>100</update_rate>
+      <visualize>true</visualize>
+      <imu>
+        <angular_velocity>
+          <x>
+            <noise type="gaussian">
+              <mean>0.0</mean>
+              <stddev>2e-4</stddev>
+              <bias_mean>0.0000075</bias_mean>
+              <bias_stddev>0.0000008</bias_stddev>
+            </noise>
+          </x>
+          <y>
+            <noise type="gaussian">
+              <mean>0.0</mean>
+              <stddev>2e-4</stddev>
+              <bias_mean>0.0000075</bias_mean>
+              <bias_stddev>0.0000008</bias_stddev>
+            </noise>
+          </y>
+          <z>
+            <noise type="gaussian">
+              <mean>0.0</mean>
+              <stddev>2e-4</stddev>
+              <bias_mean>0.0000075</bias_mean>
+              <bias_stddev>0.0000008</bias_stddev>
+            </noise>
+          </z>
+        </angular_velocity>
+        <linear_acceleration>
+          <x>
+            <noise type="gaussian">
+              <mean>0.0</mean>
+              <stddev>1.7e-2</stddev>
+              <bias_mean>0.1</bias_mean>
+              <bias_stddev>0.001</bias_stddev>
+            </noise>
+          </x>
+          <y>
+            <noise type="gaussian">
+              <mean>0.0</mean>
+              <stddev>1.7e-2</stddev>
+              <bias_mean>0.1</bias_mean>
+              <bias_stddev>0.001</bias_stddev>
+            </noise>
+          </y>
+          <z>
+            <noise type="gaussian">
+              <mean>0.0</mean>
+              <stddev>1.7e-2</stddev>
+              <bias_mean>0.1</bias_mean>
+              <bias_stddev>0.001</bias_stddev>
+            </noise>
+          </z>
+        </linear_acceleration>
+      </imu>
+    </sensor>
+  </gazebo>
+  <!-- <gazebo>
+    <plugin name="imu_plugin" filename="libgazebo_ros_imu.so">
+      <alwaysOn>true</alwaysOn>
+      <bodyName>base_footprint</bodyName>
+      <topicName>/imu_plugin/out</topicName>
+      <serviceName>imu_service</serviceName>
+      <gaussianNoise>0.0</gaussianNoise>
+      <updateRate>20.0</updateRate>
+    </plugin>
+  </gazebo> -->
+  <!-- <gazebo>
+    <plugin name="diff_drive" filename="libgazebo_ros_diff_drive.so">
+        <left_joint>left_wheel_joint</left_joint>
+        <right_joint>right_wheel_joint</right_joint>
+        <wheel_separation>0.297</wheel_separation>
+        <wheel_diameter>0.066</wheel_diameter>
+        <max_wheel_torque>200</max_wheel_torque>
+        <max_wheel_acceleration>10.0</max_wheel_acceleration>
+        <odometry_frame>odom</odometry_frame>
+        <robot_base_frame>base_link</robot_base_frame>
+        <publish_odom>true</publish_odom>
+        <publish_odom_tf>true</publish_odom_tf>
+        <publish_wheel_tf>true</publish_wheel_tf>
+    </plugin>
+</gazebo> -->
   <gazebo>
     <plugin name='diff_drive' filename='libgazebo_ros_diff_drive.so'>
@@ -73,29 +238,29 @@
       <publish_odom_tf>true</publish_odom_tf>
       <publish_wheel_tf>true</publish_wheel_tf>
-         <!-- <ros>
-        <namespace>/demo</namespace>
-        <remapping>cmd_vel:=cmd_demo</remapping>
-        <remapping>odom:=odom_demo</remapping>
-      </ros> -->
+      <!-- <ros>
+   <namespace>/demo</namespace>
+   <remapping>cmd_vel:=cmd_demo</remapping>
+   <remapping>odom:=odom_demo</remapping>
+ </ros> -->
       <!-- <updateRate>100.0</updateRate>
-      <robotNamespace>/</robotNamespace>
-      <leftFrontJoint>wheel_front_left_joint</leftFrontJoint>
-      <rightFrontJoint>wheel_front_right_joint</rightFrontJoint>
-      <leftRearJoint>wheel_back_left_joint</leftRearJoint>
-      <rightRearJoint>wheel_back_right_joint</rightRearJoint>
-      <wheelSeparation>${wheel_base}</wheelSeparation>
-      <wheelDiameter>${wheel_radius*2}</wheelDiameter>
-      <robotBaseFrame>base_link</robotBaseFrame>
-      <torque>20</torque>
-      <topicName>cmd_vel</topicName>
-      <broadcastTF>true</broadcastTF>
-      <num_wheel_pairs>2</num_wheel_pairs>
-      <max_wheel_torque>20</max_wheel_torque>
-      <max_wheel_acceleration>1.0</max_wheel_acceleration>
-      <odometry_frame>odom</odometry_frame>
-      <robot_base_frame>base_link</robot_base_frame>
-      <publish_odom>true</publish_odom>
-      <publish_odom_tf>true</publish_odom_tf>
-      <publish_wheel_tf>true</publish_wheel_tf> -->
+ <robotNamespace>/</robotNamespace>
+ <leftFrontJoint>wheel_front_left_joint</leftFrontJoint>
+ <rightFrontJoint>wheel_front_right_joint</rightFrontJoint>
+ <leftRearJoint>wheel_back_left_joint</leftRearJoint>
+ <rightRearJoint>wheel_back_right_joint</rightRearJoint>
+ <wheelSeparation>${wheel_base}</wheelSeparation>
+ <wheelDiameter>${wheel_radius*2}</wheelDiameter>
+ <robotBaseFrame>base_link</robotBaseFrame>
+ <torque>20</torque>
+ <topicName>cmd_vel</topicName>
+ <broadcastTF>true</broadcastTF>
+ <num_wheel_pairs>2</num_wheel_pairs>
+ <max_wheel_torque>20</max_wheel_torque>
+ <max_wheel_acceleration>1.0</max_wheel_acceleration>
+ <odometry_frame>odom</odometry_frame>
+ <robot_base_frame>base_link</robot_base_frame>
+ <publish_odom>true</publish_odom>
+ <publish_odom_tf>true</publish_odom_tf>
+ <publish_wheel_tf>true</publish_wheel_tf> -->
     </plugin>
   </gazebo>

File: src/deepdrive_description/urdf/wheels.xacro (robot description, xacro)
@@ -10,4 +10,6 @@
             <origin xyz="${wheel_front_offset/2 + (fb * (wheel_base / 2))} ${-lr * wheel_base/2} 0.0" rpy="0 0 ${lr*1.57}"/>
             <axis xyz="${lr} 0 0"/>
+            <!-- limit effort="1" velocity="1"/>
+            <joint_properties damping="1.0" friction="1.0"/ -->
         </joint>
         <link name="wheel_${name}_link">
@@ -48,10 +50,10 @@
                 <material name="black"/>
             </visual>
-            <collision>
+            <!-- <collision>
                 <origin xyz="0 0 0" rpy="${pi/2} 0 ${pi/2}"/>
                 <geometry>
-                    <cylinder length="${wheel_thickness}" radius="${wheel_radius}"/>
+                    <cylinder length="${wheel_thickness/2}" radius="${wheel_radius/2}"/>
                 </geometry>
-            </collision>
+            </collision> -->
             <inertial>
                 <origin xyz="0 0 0" />

Commit message: Gazebo working with ros_control

File: src/deepdrive_description/urdf/deepdrive_deepdrive.xacro (robot description, xacro)
@@ -55,13 +55,13 @@
   <xacro:include filename="$(find deepdrive_description)/urdf/lidar.xacro" />
   <xacro:include filename="$(find deepdrive_description)/urdf/camera.xacro" />
-  <!-- <ros2_control name="GazeboSystem" type="system">
+  <ros2_control name="GazeboSystem" type="system">
     <hardware>
       <plugin>gazebo_ros2_control/GazeboSystem</plugin>
-    </hardware> -->
+    </hardware>
   <!-- <hardware>
       <plugin>mock_components/GenericSystem</plugin>
       <param name="calculate_dynamics">true</param>
     </hardware> -->
-  <!-- <joint name="wheel_front_left_joint">
+  <joint name="wheel_front_left_joint">
       <command_interface name="velocity">
         <param name="min">-10</param>
@@ -95,5 +95,5 @@
       <state_interface name="position" />
     </joint>
-  </ros2_control> -->
+  </ros2_control>
   <!-- <ros2_control name="${name}" type="system">
     <xacro:unless value="${use_mock_hardware}">
@@ -121,7 +121,26 @@
     </joint>
   </ros2_control> -->
-  <!-- <gazebo>
+  <gazebo>
     <plugin filename="libgazebo_ros2_control.so" name="gazebo_ros2_control">
       <parameters>$(find deepdrive_description)/config/controllers.yaml</parameters>
+    </plugin>
+  </gazebo>
+<!-- This one works in gazebo -->
+  <!-- <gazebo>
+    <plugin name='diff_drive' filename='libgazebo_ros_diff_drive.so'>
+      <num_wheel_pairs>2</num_wheel_pairs>
+      <left_joint>wheel_front_left_joint</left_joint>
+      <right_joint>wheel_front_right_joint</right_joint>
+      <left_joint>wheel_back_left_joint</left_joint>
+      <right_joint>wheel_back_right_joint</right_joint>
+      <wheel_separation>${wheel_base}</wheel_separation>
+      <wheel_diameter>${wheel_radius*2}</wheel_diameter>
+      <max_wheel_torque>200</max_wheel_torque>
+      <max_wheel_acceleration>10.0</max_wheel_acceleration>
+      <odometry_frame>odom</odometry_frame>
+      <robot_base_frame>base_footprint</robot_base_frame>
+      <publish_odom>true</publish_odom>
+      <publish_odom_tf>true</publish_odom_tf>
+      <publish_wheel_tf>true</publish_wheel_tf>
     </plugin>
   </gazebo> -->
@@ -194,74 +213,3 @@
     </sensor>
   </gazebo>
-  <!-- <gazebo>
-    <plugin name="imu_plugin" filename="libgazebo_ros_imu.so">
-      <alwaysOn>true</alwaysOn>
-      <bodyName>base_footprint</bodyName>
-      <topicName>/imu_plugin/out</topicName>
-      <serviceName>imu_service</serviceName>
-      <gaussianNoise>0.0</gaussianNoise>
-      <updateRate>20.0</updateRate>
-    </plugin>
-  </gazebo> -->
-  <!-- <gazebo>
-    <plugin name="diff_drive" filename="libgazebo_ros_diff_drive.so">
-        <left_joint>left_wheel_joint</left_joint>
-        <right_joint>right_wheel_joint</right_joint>
-        <wheel_separation>0.297</wheel_separation>
-        <wheel_diameter>0.066</wheel_diameter>
-        <max_wheel_torque>200</max_wheel_torque>
-        <max_wheel_acceleration>10.0</max_wheel_acceleration>
-        <odometry_frame>odom</odometry_frame>
-        <robot_base_frame>base_link</robot_base_frame>
-        <publish_odom>true</publish_odom>
-        <publish_odom_tf>true</publish_odom_tf>
-        <publish_wheel_tf>true</publish_wheel_tf>
-    </plugin>
-</gazebo> -->
-  <gazebo>
-    <plugin name='diff_drive' filename='libgazebo_ros_diff_drive.so'>
-      <!-- Wheel Information -->
-      <num_wheel_pairs>2</num_wheel_pairs>
-      <left_joint>wheel_front_left_joint</left_joint>
-      <right_joint>wheel_front_right_joint</right_joint>
-      <left_joint>wheel_back_left_joint</left_joint>
-      <right_joint>wheel_back_right_joint</right_joint>
-      <wheel_separation>${wheel_base}</wheel_separation>
-      <wheel_diameter>${wheel_radius*2}</wheel_diameter>
-      <!-- Limits -->
-      <max_wheel_torque>200</max_wheel_torque>
-      <max_wheel_acceleration>10.0</max_wheel_acceleration>
-      <!-- Output -->
-      <odometry_frame>odom</odometry_frame>
-      <robot_base_frame>base_footprint</robot_base_frame>
-      <publish_odom>true</publish_odom>
-      <publish_odom_tf>true</publish_odom_tf>
-      <publish_wheel_tf>true</publish_wheel_tf>
-      <!-- <ros>
-   <namespace>/demo</namespace>
-   <remapping>cmd_vel:=cmd_demo</remapping>
-   <remapping>odom:=odom_demo</remapping>
- </ros> -->
-      <!-- <updateRate>100.0</updateRate>
- <robotNamespace>/</robotNamespace>
- <leftFrontJoint>wheel_front_left_joint</leftFrontJoint>
- <rightFrontJoint>wheel_front_right_joint</rightFrontJoint>
- <leftRearJoint>wheel_back_left_joint</leftRearJoint>
- <rightRearJoint>wheel_back_right_joint</rightRearJoint>
- <wheelSeparation>${wheel_base}</wheelSeparation>
- <wheelDiameter>${wheel_radius*2}</wheelDiameter>
- <robotBaseFrame>base_link</robotBaseFrame>
- <torque>20</torque>
- <topicName>cmd_vel</topicName>
- <broadcastTF>true</broadcastTF>
- <num_wheel_pairs>2</num_wheel_pairs>
- <max_wheel_torque>20</max_wheel_torque>
- <max_wheel_acceleration>1.0</max_wheel_acceleration>
- <odometry_frame>odom</odometry_frame>
- <robot_base_frame>base_link</robot_base_frame>
- <publish_odom>true</publish_odom>
- <publish_odom_tf>true</publish_odom_tf>
- <publish_wheel_tf>true</publish_wheel_tf> -->
-    </plugin>
-  </gazebo>
 </robot>

File: src/deepdrive_description/urdf/wheels.xacro (robot description, xacro)
@@ -10,7 +10,15 @@
             <origin xyz="${wheel_front_offset/2 + (fb * (wheel_base / 2))} ${-lr * wheel_base/2} 0.0" rpy="0 0 ${lr*1.57}"/>
             <axis xyz="${lr} 0 0"/>
-            <!-- limit effort="1" velocity="1"/>
-            <joint_properties damping="1.0" friction="1.0"/ -->
+            <!-- <dynamics damping="0.8"/> -->
+            <!-- <limit effort="100" velocity="0.5"/> -->
         </joint>
+        <!-- <joint name="${prefix}right_wheel_joint" type="continuous">
+            <parent link="${prefix}base_link"/>
+            <child link="${prefix}right_wheel"/>
+            <origin xyz="0 ${base_width/2} ${z_offset}" rpy="0 0 0"/>
+            <axis xyz="0 1 0"/>
+            <dynamics damping="0.2"/>
+            <limit effort="100" velocity="1.0"/>
+        </joint> -->
         <link name="wheel_${name}_link">
             <visual>
@@ -29,5 +37,5 @@
             <inertial>
                 <origin xyz="0 0 0" />
-                <mass value="2.8498940e-02" />
+                <mass value=".05" />
                 <inertia ixx="1.1175580e-05" ixy="-4.2369783e-11" ixz="-5.9381719e-09" iyy="1.1192413e-05" iyz="-1.4400107e-11" izz="2.0712558e-05" />
             </inertial>
@@ -65,4 +73,12 @@
             <material>Gazebo/Black</material>
         </gazebo>
+        <!-- Friction coefficients -->
+        <gazebo reference="wheel_${name}_link">
+            <mu1 value="0.02"/>
+            <mu2 value="0.02"/>
+            <!-- <kp value="10000000.0" />
+            <kd value="1.0" />
+            <fdir1 value="1 0 0"/> -->
+        </gazebo>
     </xacro:macro>
 </robot>

Commit message: Pointcloud working

File: src/deepdrive_description/urdf/deepdrive_deepdrive.xacro (robot description, xacro)
@@ -47,9 +47,8 @@
   </joint>
   <link name="imu_link"/>
-  <!--
-   <joint name="oak_joint" type="fixed">
+   <!-- <joint name="oak_joint" type="fixed">
     <parent link="base_link"/>
     <child link="oak"/>
-    <origin xyz="0.0 0 0.068" rpy="0 0 1.57"/>
+    <origin xyz="0.0 0 0.068" rpy="0 0 0"/>
   </joint>
   <link name="oak"/> -->

File: src/deepdrive_description/urdf/lidar.xacro (robot description, xacro)
@@ -29,5 +29,5 @@
         <parent link="base_scan"/>
         <child link="laser"/>
-        <origin xyz="0.0 0 0.058" rpy="0 0 1.57"/>
+        <origin xyz="0.0 0 0.058" rpy="0 0 ${pi}"/>
     </joint>
     <link name="laser"/>

File: src/deepdrive_description/urdf/oakdlite.xacro (robot description, xacro)
@@ -31,5 +31,5 @@
     <!-- RGB -->
     <joint name="${mount_point}_optical_joint" type="fixed">
-      <origin xyz="0 0 0" rpy="${-pi/2} 0 ${-pi/2}"/>
+      <origin xyz="0.1 0 0.2" rpy="${-pi/2} 0 ${-pi/2}"/>
       <parent link="${mount_point}"/>
       <child link="${mount_point}_optical_frame"/>

Commit message: localization looking better

File: src/deepdrive_description/urdf/deepdrive_deepdrive.xacro (robot description, xacro)
@@ -49,8 +49,8 @@
    <!-- <joint name="oak_joint" type="fixed">
     <parent link="base_link"/>
-    <child link="oak"/>
-    <origin xyz="0.0 0 0.068" rpy="0 0 0"/>
-  </joint>
-  <link name="oak"/> -->
+    <child link="camera_depth_imu_frame"/>
+    <origin xyz="0.0 0 0.0" rpy="0 0 0"/>
+  </joint> -->
+  <!-- <link name="camera_depth_imu_frame"/> -->
   <!-- LIDAR -->
   <xacro:include filename="$(find deepdrive_description)/urdf/lidar.xacro" />
@@ -67,5 +67,5 @@
     </joint>
   </xacro:macro>
-  <ros2_control name="GazeboSystem" type="system">
+  <ros2_control name="deepdrive" type="system">
     <!-- Gazebo simulation -->
     <xacro:if value="$(arg sim_mode)">

Commit message: Working on ros2

File: src/deepdrive_description/urdf/deepdrive_deepdrive.xacro (robot description, xacro)
@@ -56,55 +56,7 @@
   <xacro:include filename="$(find deepdrive_description)/urdf/lidar.xacro" />
   <xacro:include filename="$(find deepdrive_description)/urdf/camera.xacro" />
-  <!-- ros2_control -->
-  <xacro:macro name="ros2_wheel_joint" params="name">
-    <joint name="wheel_${name}_joint">
-      <command_interface name="velocity">
-        <param name="min">-1</param>
-        <param name="max">1</param>
-      </command_interface>
-      <state_interface name="position" />
-      <state_interface name="velocity" />
-    </joint>
-  </xacro:macro>
-  <ros2_control name="deepdrive" type="system">
-    <!-- Gazebo simulation -->
-    <xacro:if value="$(arg sim_mode)">
-      <hardware>
-        <plugin>gazebo_ros2_control/GazeboSystem</plugin>
-      </hardware>
-    </xacro:if>
-    <!-- Physical Robot -->
-    <xacro:unless value="$(arg sim_mode)">
-      <hardware>
-        <plugin>deepdrive_control/DeepdriveSystemHardware</plugin>
-        <param name="mock_hardware">false</param>
-        <param name="use_wheel_encoder">true</param>
-        <param name="encoder_ticks_per_rev">20</param>
-        <param name="pin_left_enable">32</param>
-        <param name="pin_left_forward">38</param>
-        <param name="pin_left_backward">37</param>
-        <param name="pin_left_encoder">11</param>
-        <param name="pin_right_enable">33</param>
-        <param name="pin_right_forward">35</param>
-        <param name="pin_right_backward">36</param>
-        <param name="pin_right_encoder">12</param>
-        <param name="pwm_hz">50</param>
-        <!-- should match controller.yaml update rate -->
-        <param name="command_rate">50</param>
-      </hardware>
-    </xacro:unless>
-    <xacro:ros2_wheel_joint name="back_right" />
-    <xacro:ros2_wheel_joint name="front_left" />
-    <xacro:ros2_wheel_joint name="back_left" />
-    <xacro:ros2_wheel_joint name="front_right" />
-  </ros2_control>
   <xacro:if value="$(arg sim_mode)">
+    <!-- This one works in gazebo without ros2_control -->
     <gazebo>
-      <plugin filename="libgazebo_ros2_control.so" name="gazebo_ros2_control">
-        <parameters>$(find deepdrive_description)/config/controllers.yaml</parameters>
-      </plugin>
-    </gazebo>
-    <!-- This one works in gazebo without ros2_control -->
-    <!-- <gazebo>
     <plugin name='diff_drive' filename='libgazebo_ros_diff_drive.so'>
       <num_wheel_pairs>2</num_wheel_pairs>
@@ -123,5 +75,5 @@
       <publish_wheel_tf>true</publish_wheel_tf>
     </plugin>
-  </gazebo> -->
+  </gazebo>
     <gazebo reference="imu_link">
       <sensor name="imu_sensor" type="imu">
