Commit message: About to retry again with cpp node

File: src/deepdrive_description/urdf/deepdrive_deepdrive.xacro (robot description, xacro)
@@ -5,5 +5,5 @@
   <xacro:property name="wheel_base" value="0.175" />
   <xacro:property name="wheel_radius" value="0.035" />
-  <!-- <xacro:property name="use_mock_hardware" value="0.035" /> -->
+  <!-- <xacro:property name="use_mock_hardware" value="true" /> -->
   <xacro:include filename="$(find deepdrive_description)/urdf/common_properties.xacro"/>
   <xacro:include filename="$(find deepdrive_description)/urdf/wheels.xacro"/>
@@ -56,15 +56,4 @@
   <xacro:include filename="$(find deepdrive_description)/urdf/lidar.xacro" />
   <xacro:include filename="$(find deepdrive_description)/urdf/camera.xacro" />
-  <!-- ros2_control -->
-  <xacro:macro name="ros2_wheel_joint" params="name">
-    <joint name="wheel_${name}_joint">
-      <command_interface name="velocity">
-        <param name="min">-1</param>
-        <param name="max">1</param>
-      </command_interface>
-      <state_interface name="position" />
-      <state_interface name="velocity" />
-    </joint>
-  </xacro:macro>
   <xacro:if value="$(arg sim_mode)">
     <gazebo>

Commit message: Sonar working

File: src/deepdrive_description/urdf/deepdrive_deepdrive.xacro (robot description, xacro)
@@ -72,9 +72,22 @@
     <parent link="base_link"/>
     <child link="ldlidar_base"/>
-    <origin xyz="-0.05 0.001 0.120" rpy="0 0 0"/>
+    <origin xyz="-0.05 0.001 0.150" rpy="0 0 0"/>
   </joint>
   <!-- <link name="imu_link"/> -->
   <xacro:include filename="$(find deepdrive_description)/urdf/lidar.xacro" />
   <xacro:include filename="$(find deepdrive_description)/urdf/camera.xacro" />
+  <!-- Ultrasonic Sonar -->
+  <joint name="sonar_front_joint" type="fixed">
+    <parent link="base_link"/>
+    <child link="sonar_front_link"/>
+    <origin xyz="0.125 0.0 0.0" rpy="0 0 0"/>
+  </joint>
+  <link name="sonar_front_link"/>
+  <joint name="sonar_back_joint" type="fixed">
+    <parent link="base_link"/>
+    <child link="sonar_back_link"/>
+    <origin xyz="-0.25 0.0 0.0" rpy="0 0 ${pi}"/>
+  </joint>
+  <link name="sonar_back_link"/>
   <xacro:if value="$(arg sim_mode)">
     <!-- This one works in gazebo without ros2_control -->

Commit message: Added v5 meshes

File: src/deepdrive_description/urdf/deepdrive_deepdrive.xacro (robot description, xacro)
@@ -3,6 +3,6 @@
   xmlns:xacro="http://ros.org/wiki/xacro">
   <xacro:arg name="sim_mode" default="false"/>
-  <xacro:property name="wheel_base" value="0.24" />
-  <xacro:property name="wheel_radius" value="0.0445" />
+  <xacro:property name="wheel_base" value="0.32385" />
+  <xacro:property name="wheel_radius" value="0.08" />
   <!-- <xacro:property name="use_mock_hardware" value="true" /> -->
   <xacro:include filename="$(find deepdrive_description)/urdf/common_properties.xacro"/>

File: src/deepdrive_description/urdf/lidar.xacro (robot description, xacro)
@@ -5,5 +5,5 @@
             <origin xyz="0 0 0" rpy="0 0 0"/>
             <geometry>
-                <mesh filename="package://ldlidar_node/urdf/model/LD19.stl" scale="0.001 0.001 0.001" />
+                <mesh filename="package://deepdrive_description/meshes/sensors/ld19.stl" scale="0.001 0.001 0.001" />
             </geometry>
             <material name="ldlidar_mat">

Commit message: updating deepdrive_description

File: src/deepdrive_description/urdf/deepdrive_deepdrive.xacro (robot description, xacro)
@@ -1,36 +1,39 @@
-<?xml version="1.0" ?>
+<?xml version="1.0"?>
 <robot name="deepdrive_deepdrive"
   xmlns:xacro="http://ros.org/wiki/xacro">
-  <xacro:arg name="sim_mode" default="false"/>
-  <xacro:property name="wheel_base" value="0.32385" />
+  <xacro:arg name="sim_mode" default="false" />
+  <xacro:property name="wheel_base" value="0.26" />
   <xacro:property name="wheel_radius" value="0.08" />
   <!-- <xacro:property name="use_mock_hardware" value="true" /> -->
-  <xacro:include filename="$(find deepdrive_description)/urdf/common_properties.xacro"/>
-  <xacro:include filename="$(find deepdrive_description)/urdf/wheels.xacro"/>
-  <link name="base_footprint"/>
+  <xacro:include filename="$(find deepdrive_description)/urdf/common_properties.xacro" />
+  <xacro:include filename="$(find deepdrive_description)/urdf/wheels.xacro" />
+  <xacro:include filename="$(find deepdrive_description)/urdf/sonar.xacro" />
+  <link name="base_footprint" />
   <joint name="base_joint" type="fixed">
-    <parent link="base_footprint"/>
+    <parent link="base_footprint" />
     <child link="base_link" />
-    <origin xyz="0 0 0.010" rpy="0 0 0"/>
+    <origin xyz="0 0 0.010" rpy="0 0 0" />
   </joint>
   <!-- Frame/Chassis -->
   <link name="base_link">
     <visual>
-      <origin xyz="-0.064 0 0.0" rpy="0 0 ${pi/2}"/>
-      <geometry>
-        <mesh filename="package://deepdrive_description/meshes/bases/chassis.stl" scale=".001 .001 .001"/>
-      </geometry>
-      <material name="dark"/>
+      <origin xyz="-0.064 0 0.0" rpy="0 0 ${3*pi/2}" />
+      <geometry>
+        <mesh filename="package://deepdrive_description/meshes/bases/chassis.stl"
+          scale=".001 .001 .001" />
+      </geometry>
+      <material name="black" />
     </visual>
     <collision>
-      <origin xyz="-0.064 0 0.047" rpy="0 0 0"/>
-      <geometry>
-        <box size="0.310 0.140 0.120"/>
+      <origin xyz="-0.064 0 0.047" rpy="0 0 0" />
+      <geometry>
+        <box size="0.310 0.140 0.120" />
       </geometry>
     </collision>
     <inertial>
-      <origin xyz="0 0 0" rpy="0 0 0"/>
-      <mass value="2.3729096e+00"/>
-      <inertia ixx="8.7002718e-03" ixy="-4.7576583e-05" ixz="1.1160499e-04" iyy="8.6195418e-03" iyz="-3.5422299e-06" izz="1.4612727e-02" />
+      <origin xyz="0 0 0" rpy="0 0 0" />
+      <mass value="2.3729096e+00" />
+      <inertia ixx="8.7002718e-03" ixy="-4.7576583e-05" ixz="1.1160499e-04" iyy="8.6195418e-03"
+        iyz="-3.5422299e-06" izz="1.4612727e-02" />
     </inertial>
   </link>
@@ -40,54 +43,85 @@
   <!-- Body-->
   <joint name="body_joint" type="fixed">
-    <parent link="base_link"/>
+    <parent link="base_link" />
     <child link="body_link" />
-    <origin xyz="0 0 0.0" rpy="0 0 0"/>
+    <origin xyz="0 0 0.0" rpy="0 0 0" />
   </joint>
   <link name="body_link">
     <visual>
-      <origin xyz="-0.064 0 0.0" rpy="0 0 ${pi/2}"/>
-      <geometry>
-        <mesh filename="package://deepdrive_description/meshes/bases/body.stl" scale=".001 .001 .001"/>
-      </geometry>
-      <material name="black"/>
-    </visual>
-  </link>
-  <gazebo reference="base_link">
+      <origin xyz="-0.064 0 0.001" rpy="0 0 ${3*pi/2}" />
+      <geometry>
+        <mesh filename="package://deepdrive_description/meshes/bases/body.stl"
+          scale=".001 .001 .001" />
+      </geometry>
+      <material name="red" />
+    </visual>
+  </link>
+  <gazebo reference="body_link">
+    <material>Gazebo/Red</material>
+  </gazebo>
+  <!-- Wheels -->
+  <xacro:wheel name="front_right" lr="1" fb="1" wheel_base="${wheel_base}"
+    wheel_radius="${wheel_radius}" />
+  <xacro:wheel name="back_right" lr="1" fb="-1" wheel_base="${wheel_base}"
+    wheel_radius="${wheel_radius}" />
+  <xacro:wheel name="front_left" lr="-1" fb="1" wheel_base="${wheel_base}"
+    wheel_radius="${wheel_radius}" />
+  <xacro:wheel name="back_left" lr="-1" fb="-1" wheel_base="${wheel_base}"
+    wheel_radius="${wheel_radius}" />
+  <!-- IMU -->
+  <joint name="imu_joint" type="fixed">
+    <parent link="base_link" />
+    <child link="imu_link" />
+    <origin xyz="0.12 0 0.111" rpy="0 0 0" />
+  </joint>
+  <link name="imu_link">
+    <visual>
+      <origin xyz="0 0 0" rpy="0 0 -${pi/2}" />
+      <!-- <origin xyz=".325 0 -.07" rpy="0 0 0" /> -->
+      <geometry>
+        <mesh filename="package://deepdrive_description/meshes/sensors/imu.stl"
+          scale=".001 .001 .001" />
+      </geometry>
+      <material name="white" />
+    </visual>
+  </link>
+  <!-- LIDAR -->
+  <joint name="ldlidar_joint" type="fixed">
+    <parent link="base_link" />
+    <child link="ldlidar_base" />
+    <origin xyz="-0.119 0.0009 0.118" rpy="0 0 0" />
+  </joint>
+  <xacro:include filename="$(find deepdrive_description)/urdf/lidar.xacro" />
+  <!-- Oak-d-lite Camera -->
+  <xacro:include filename="$(find deepdrive_description)/urdf/oakdlite.xacro" />
+  <joint name="base_camera_depth_joint" type="fixed">
+    <parent link="base_link" />
+    <child link="camera_depth" />
+    <origin xyz="0.295 0 0.08" rpy="0 0 0" />
+  </joint>
+  <link name="camera_depth" />
+  <xacro:camera_depth mount_point="camera_depth" />
+  <!-- Ultrasonic Sonar -->
+  <xacro:sonar name="front_right" xyz=".296 .064 .035" rpy="0 0 ${5*pi/180}" />
+  <xacro:sonar name="front_left" xyz=".296 -.064 .035" rpy="0 0 -${5*pi/180}" />
+  <!-- Speaker -->
+  <joint name="speaker_joint" type="fixed">
+    <parent link="base_link" />
+    <child link="speaker_link" />
+    <origin xyz="-.03 0 0.1" rpy="0 0 0" />
+  </joint>
+  <link name="speaker_link">
+    <visual>
+      <origin xyz="0 -0.41 0" rpy="0 0 0" />
+      <geometry>
+        <mesh filename="package://deepdrive_description/meshes/sensors/speaker.stl"
+          scale=".001 .001 .001" />
+      </geometry>
+      <material name="black" />
+    </visual>
+  </link>
+  <gazebo reference="speaker_link">
     <material>Gazebo/Black</material>
   </gazebo>
-  <!-- Wheels -->
-  <xacro:wheel name="front_right" lr="1" fb="1" wheel_base="${wheel_base}" wheel_radius="${wheel_radius}" />
-  <xacro:wheel name="back_right" lr="1" fb="-1" wheel_base="${wheel_base}" wheel_radius="${wheel_radius}" />
-  <xacro:wheel name="front_left" lr="-1" fb="1" wheel_base="${wheel_base}" wheel_radius="${wheel_radius}" />
-  <xacro:wheel name="back_left" lr="-1" fb="-1" wheel_base="${wheel_base}" wheel_radius="${wheel_radius}" />
-  <!-- IMU -->
-  <joint name="imu_joint" type="fixed">
-    <parent link="base_link"/>
-    <child link="imu_link"/>
-    <origin xyz="0.0 0 0.068" rpy="0 0 0"/>
-  </joint>
-  <link name="imu_link"/>
-  <!-- LIDAR -->
-  <joint name="ldlidar_joint" type="fixed">
-    <parent link="base_link"/>
-    <child link="ldlidar_base"/>
-    <origin xyz="-0.05 0.001 0.150" rpy="0 0 0"/>
-  </joint>
-  <!-- <link name="imu_link"/> -->
-  <xacro:include filename="$(find deepdrive_description)/urdf/lidar.xacro" />
-  <xacro:include filename="$(find deepdrive_description)/urdf/camera.xacro" />
-  <!-- Ultrasonic Sonar -->
-  <joint name="sonar_front_joint" type="fixed">
-    <parent link="base_link"/>
-    <child link="sonar_front_link"/>
-    <origin xyz="0.125 0.0 0.0" rpy="0 0 0"/>
-  </joint>
-  <link name="sonar_front_link"/>
-  <joint name="sonar_back_joint" type="fixed">
-    <parent link="base_link"/>
-    <child link="sonar_back_link"/>
-    <origin xyz="-0.25 0.0 0.0" rpy="0 0 ${pi}"/>
-  </joint>
-  <link name="sonar_back_link"/>
   <xacro:if value="$(arg sim_mode)">
     <!-- This one works in gazebo without ros2_control -->

File: src/deepdrive_description/urdf/wheels.xacro (robot description, xacro)
@@ -3,5 +3,5 @@
     xmlns:xacro="http://ros.org/wiki/xacro">
     <xacro:property name="wheel_thickness" value="0.025" />
-    <xacro:property name="wheel_front_offset" value="-.13" />
+    <xacro:property name="wheel_front_offset" value=".13" />
     <xacro:macro name="wheel" params="lr fb name wheel_base wheel_radius">
         <joint name="wheel_${name}_joint" type="continuous">

Commit message: fixed up odom

File: src/deepdrive_description/urdf/deepdrive_deepdrive.xacro (robot description, xacro)
@@ -70,10 +70,10 @@
     wheel_radius="${wheel_radius}" />
   <!-- IMU -->
-  <joint name="imu_joint" type="fixed">
-    <parent link="base_link" />
-    <child link="imu_link" />
+  <joint name="imu_base_joint" type="fixed">
+    <parent link="base_link" />
+    <child link="imu_base_link" />
     <origin xyz="0.12 0 0.111" rpy="0 0 0" />
   </joint>
-  <link name="imu_link">
+  <link name="imu_base_link">
     <visual>
       <origin xyz="0 0 0" rpy="0 0 -${pi/2}" />
@@ -86,4 +86,10 @@
     </visual>
   </link>
+  <joint name="imu_joint" type="fixed">
+    <parent link="imu_base_link" />
+    <child link="imu_link" />
+    <origin xyz="0 0 0" rpy="${pi/2} 0 ${pi}" />
+  </joint>
+  <link name="imu_link"></link>
   <!-- LIDAR -->
   <joint name="ldlidar_joint" type="fixed">

Commit message: Switched back to ros2_control

File: src/deepdrive_description/urdf/deepdrive_deepdrive.xacro (robot description, xacro)
@@ -3,10 +3,13 @@
   xmlns:xacro="http://ros.org/wiki/xacro">
   <xacro:arg name="sim_mode" default="false" />
+  <xacro:arg name="use_ros2_control" default="true" />
   <xacro:property name="wheel_base" value="0.26" />
   <xacro:property name="wheel_radius" value="0.08" />
-  <!-- <xacro:property name="use_mock_hardware" value="true" /> -->
+  <xacro:property name="use_mock_hardware" value="false" />
   <xacro:include filename="$(find deepdrive_description)/urdf/common_properties.xacro" />
   <xacro:include filename="$(find deepdrive_description)/urdf/wheels.xacro" />
   <xacro:include filename="$(find deepdrive_description)/urdf/sonar.xacro" />
+  <xacro:include filename="$(find deepdrive_description)/urdf/optical_flow.xacro" />
+  <xacro:include filename="$(find deepdrive_description)/urdf/ros2_control.xacro" />
   <link name="base_footprint" />
   <joint name="base_joint" type="fixed">
@@ -20,6 +23,5 @@
       <origin xyz="-0.064 0 0.0" rpy="0 0 ${3*pi/2}" />
       <geometry>
-        <mesh filename="package://deepdrive_description/meshes/bases/chassis.stl"
-          scale=".001 .001 .001" />
+        <mesh filename="package://deepdrive_description/meshes/bases/chassis.stl" scale=".001 .001 .001" />
       </geometry>
       <material name="black" />
@@ -34,6 +36,5 @@
       <origin xyz="0 0 0" rpy="0 0 0" />
       <mass value="2.3729096e+00" />
-      <inertia ixx="8.7002718e-03" ixy="-4.7576583e-05" ixz="1.1160499e-04" iyy="8.6195418e-03"
-        iyz="-3.5422299e-06" izz="1.4612727e-02" />
+      <inertia ixx="8.7002718e-03" ixy="-4.7576583e-05" ixz="1.1160499e-04" iyy="8.6195418e-03" iyz="-3.5422299e-06" izz="1.4612727e-02" />
     </inertial>
   </link>
@@ -51,6 +52,5 @@
       <origin xyz="-0.064 0 0.001" rpy="0 0 ${3*pi/2}" />
       <geometry>
-        <mesh filename="package://deepdrive_description/meshes/bases/body.stl"
-          scale=".001 .001 .001" />
+        <mesh filename="package://deepdrive_description/meshes/bases/body.stl" scale=".001 .001 .001" />
       </geometry>
       <material name="red" />
@@ -61,12 +61,8 @@
   </gazebo>
   <!-- Wheels -->
-  <xacro:wheel name="front_right" lr="1" fb="1" wheel_base="${wheel_base}"
-    wheel_radius="${wheel_radius}" />
-  <xacro:wheel name="back_right" lr="1" fb="-1" wheel_base="${wheel_base}"
-    wheel_radius="${wheel_radius}" />
-  <xacro:wheel name="front_left" lr="-1" fb="1" wheel_base="${wheel_base}"
-    wheel_radius="${wheel_radius}" />
-  <xacro:wheel name="back_left" lr="-1" fb="-1" wheel_base="${wheel_base}"
-    wheel_radius="${wheel_radius}" />
+  <xacro:wheel name="front_right" lr="1" fb="1" wheel_base="${wheel_base}" wheel_radius="${wheel_radius}" />
+  <xacro:wheel name="back_right" lr="1" fb="-1" wheel_base="${wheel_base}" wheel_radius="${wheel_radius}" />
+  <xacro:wheel name="front_left" lr="-1" fb="1" wheel_base="${wheel_base}" wheel_radius="${wheel_radius}" />
+  <xacro:wheel name="back_left" lr="-1" fb="-1" wheel_base="${wheel_base}" wheel_radius="${wheel_radius}" />
   <!-- IMU -->
   <joint name="imu_base_joint" type="fixed">
@@ -80,6 +76,5 @@
       <!-- <origin xyz=".325 0 -.07" rpy="0 0 0" /> -->
       <geometry>
-        <mesh filename="package://deepdrive_description/meshes/sensors/imu.stl"
-          scale=".001 .001 .001" />
+        <mesh filename="package://deepdrive_description/meshes/sensors/imu.stl" scale=".001 .001 .001" />
       </geometry>
       <material name="white" />
@@ -111,4 +106,7 @@
   <xacro:sonar name="front_right" xyz=".296 .064 .035" rpy="0 0 ${5*pi/180}" />
   <xacro:sonar name="front_left" xyz=".296 -.064 .035" rpy="0 0 -${5*pi/180}" />
+  <!-- Optical Flow -->
+  <!-- <xacro:optical_flow name="front" xyz=".296 -.064 .035" rpy="0 0 -${5*pi/180}" /> -->
+  <xacro:optical_flow name="front" xyz=".296 0 .005" rpy="0 ${pi/2} 0" />
   <!-- Speaker -->
   <joint name="speaker_joint" type="fixed">
@@ -121,6 +119,5 @@
       <origin xyz="0 -0.41 0" rpy="0 0 0" />
       <geometry>
-        <mesh filename="package://deepdrive_description/meshes/sensors/speaker.stl"
-          scale=".001 .001 .001" />
+        <mesh filename="package://deepdrive_description/meshes/sensors/speaker.stl" scale=".001 .001 .001" />
       </geometry>
       <material name="black" />
@@ -130,5 +127,10 @@
     <material>Gazebo/Black</material>
   </gazebo>
-  <xacro:if value="$(arg sim_mode)">
+  <!-- ros2_control-->
+  <xacro:if value="$(arg use_ros2_control)">
+    <xacro:deepdrive_ros2_control name="diff_drive_controller" use_mock_hardware="${use_mock_hardware}" />
+  </xacro:if>
+  <xacro:unless value="$(arg use_ros2_control)">
+    <!-- <xacro:if value="$(arg sim_mode)"> -->
     <!-- This one works in gazebo without ros2_control -->
     <gazebo>
@@ -157,72 +159,73 @@
       </plugin>
     </gazebo>
-    <gazebo reference="imu_link">
-      <sensor name="imu_sensor" type="imu">
-        <plugin filename="libgazebo_ros_imu_sensor.so" name="imu_plugin">
-          <ros>
-            <namespace>/</namespace>
-            <remapping>~/out:=imu</remapping>
-          </ros>
-          <initial_orientation_as_reference>false</initial_orientation_as_reference>
-        </plugin>
-        <always_on>true</always_on>
-        <update_rate>50</update_rate>
-        <visualize>true</visualize>
-        <imu>
-          <angular_velocity>
-            <x>
-              <noise type="gaussian">
-                <mean>0.0</mean>
-                <stddev>2e-4</stddev>
-                <bias_mean>0.0000075</bias_mean>
-                <bias_stddev>0.0000008</bias_stddev>
-              </noise>
-            </x>
-            <y>
-              <noise type="gaussian">
-                <mean>0.0</mean>
-                <stddev>2e-4</stddev>
-                <bias_mean>0.0000075</bias_mean>
-                <bias_stddev>0.0000008</bias_stddev>
-              </noise>
-            </y>
-            <z>
-              <noise type="gaussian">
-                <mean>0.0</mean>
-                <stddev>2e-4</stddev>
-                <bias_mean>0.0000075</bias_mean>
-                <bias_stddev>0.0000008</bias_stddev>
-              </noise>
-            </z>
-          </angular_velocity>
-          <linear_acceleration>
-            <x>
-              <noise type="gaussian">
-                <mean>0.0</mean>
-                <stddev>1.7e-2</stddev>
-                <bias_mean>0.1</bias_mean>
-                <bias_stddev>0.001</bias_stddev>
-              </noise>
-            </x>
-            <y>
-              <noise type="gaussian">
-                <mean>0.0</mean>
-                <stddev>1.7e-2</stddev>
-                <bias_mean>0.1</bias_mean>
-                <bias_stddev>0.001</bias_stddev>
-              </noise>
-            </y>
-            <z>
-              <noise type="gaussian">
-                <mean>0.0</mean>
-                <stddev>1.7e-2</stddev>
-                <bias_mean>0.1</bias_mean>
-                <bias_stddev>0.001</bias_stddev>
-              </noise>
-            </z>
-          </linear_acceleration>
-        </imu>
-      </sensor>
-    </gazebo>
-  </xacro:if>
+  </xacro:unless>
+  <gazebo reference="imu_link">
+    <sensor name="imu_sensor" type="imu">
+      <plugin filename="libgazebo_ros_imu_sensor.so" name="imu_plugin">
+        <ros>
+          <namespace>/</namespace>
+          <remapping>~/out:=imu</remapping>
+        </ros>
+        <initial_orientation_as_reference>false</initial_orientation_as_reference>
+      </plugin>
+      <always_on>true</always_on>
+      <update_rate>50</update_rate>
+      <visualize>true</visualize>
+      <imu>
+        <angular_velocity>
+          <x>
+            <noise type="gaussian">
+              <mean>0.0</mean>
+              <stddev>2e-4</stddev>
+              <bias_mean>0.0000075</bias_mean>
+              <bias_stddev>0.0000008</bias_stddev>
+            </noise>
+          </x>
+          <y>
+            <noise type="gaussian">
+              <mean>0.0</mean>
+              <stddev>2e-4</stddev>
+              <bias_mean>0.0000075</bias_mean>
+              <bias_stddev>0.0000008</bias_stddev>
+            </noise>
+          </y>
+          <z>
+            <noise type="gaussian">
+              <mean>0.0</mean>
+              <stddev>2e-4</stddev>
+              <bias_mean>0.0000075</bias_mean>
+              <bias_stddev>0.0000008</bias_stddev>
+            </noise>
+          </z>
+        </angular_velocity>
+        <linear_acceleration>
+          <x>
+            <noise type="gaussian">
+              <mean>0.0</mean>
+              <stddev>1.7e-2</stddev>
+              <bias_mean>0.1</bias_mean>
+              <bias_stddev>0.001</bias_stddev>
+            </noise>
+          </x>
+          <y>
+            <noise type="gaussian">
+              <mean>0.0</mean>
+              <stddev>1.7e-2</stddev>
+              <bias_mean>0.1</bias_mean>
+              <bias_stddev>0.001</bias_stddev>
+            </noise>
+          </y>
+          <z>
+            <noise type="gaussian">
+              <mean>0.0</mean>
+              <stddev>1.7e-2</stddev>
+              <bias_mean>0.1</bias_mean>
+              <bias_stddev>0.001</bias_stddev>
+            </noise>
+          </z>
+        </linear_acceleration>
+      </imu>
+    </sensor>
+  </gazebo>
+<!-- </xacro:if> -->
 </robot>

Commit message: Nav2 working

File: src/deepdrive_description/urdf/deepdrive_deepdrive.xacro (robot description, xacro)
@@ -4,5 +4,5 @@
   <xacro:arg name="sim_mode" default="false" />
   <xacro:arg name="use_ros2_control" default="true" />
-  <xacro:property name="wheel_base" value="0.26" />
+  <xacro:property name="wheel_base" value="0.328" />
   <xacro:property name="wheel_radius" value="0.08" />
   <xacro:property name="use_mock_hardware" value="false" />
