Commit message: Working on dockerfile

File: src/deepdrive_nav2_bringup/urdf/deepdrive.urdf (robot description, URDF)
Before this commit: robot deepdrive, 13 links, 12 joints
Links:
- link base_link: geometry collision box size=0.266 0.266 0.094; visual mesh filename=package://deepdrive_simulations/models/deepdrive_common/mes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 scale=0.001 0.001 0.001
- link base_scan: geometry collision cylinder length=0.0315 radius=0.055; visual mesh filename=package://deepdrive_simulations/models/deepdrive_common/mes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 scale=0.001 0.001 0.001
- link camera_link: geometry collision box size=0.012 0.132 0.020; visual mesh filename=package://deepdrive_simulations/models/deepdrive_common/mes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
- link wheel_left_link: geometry collision cylinder length=0.018 radius=0.033; visual mesh filename=package://deepdrive_simulations/models/deepdrive_common/mes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 scale=0.001 0.001 0.001
- link wheel_right_link: geometry collision cylinder length=0.018 radius=0.033; visual mesh filename=package://deepdrive_simulations/models/deepdrive_common/mes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 scale=0.001 0.001 0.001

File: src/deepdrive_simulations/deepdrive_gazebo/urdf/deepdrive_deepdrive.urdf (robot description, URDF)
Before this commit: robot deepdrive_deepdrive, 13 links, 12 joints
Links:
- link base_link: geometry collision box size=0.266 0.266 0.094; visual mesh filename=package://deepdrive_simulations/models/deepdrive_common/mes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 scale=0.001 0.001 0.001
- link base_scan: geometry collision cylinder length=0.0315 radius=0.055; visual mesh filename=package://deepdrive_simulations/models/deepdrive_common/mes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 scale=0.001 0.001 0.001
- link camera_link: geometry collision box size=0.012 0.132 0.020; visual mesh filename=package://deepdrive_simulations/models/deepdrive_common/mes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
- link wheel_left_link: geometry collision cylinder length=0.018 radius=0.033; visual mesh filename=package://deepdrive_simulations/models/deepdrive_common/mes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 scale=0.001 0.001 0.001
- link wheel_right_link: geometry collision cylinder length=0.018 radius=0.033; visual mesh filename=package://deepdrive_simulations/models/deepdrive_common/mes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 scale=0.001 0.001 0.001
